File: hardware/carrier.kicad_sch (KiCad schematic)
At the start: 49 parts, among them J2 Heltec_J2, J3 Heltec_J3, U1 MT3608

Commit message: hardware: refs end in digits (KiCad annotation)
Co-Authored-By: Claude Opus 5.5 <noreply@anthropic.com>
Parts:
- removed C_BB, C_BR: 100nF, Capacitor_SMD:C_0805_2012Metric_Pad1.18x1.45mm_HandSolder, symbol Device:C
- removed C_BULK: 220uF 10V, Capacitor_THT:CP_Radial_D6.3mm_P2.50mm, symbol Device:C_Polarized
- removed C_IN: 22uF 10V, Capacitor_SMD:C_1206_3216Metric_Pad1.33x1.80mm_HandSolder, symbol Device:C
- removed C_NFC: 100uF 10V, Capacitor_THT:CP_Radial_D6.3mm_P2.50mm, symbol Device:C_Polarized
- removed D_FLY: 1N4148W, Diode_SMD:D_SOD-123, symbol Diode:1N4148W
- removed J_BAT: BAT, Connector_JST:JST_XH_B2B-XH-A_1x02_P2.50mm_Vertical, symbol Connector_Generic:Conn_01x02
- removed J_BTN_B: BTN_B, Connector_JST:JST_XH_B4B-XH-A_1x04_P2.50mm_Vertical, symbol Connector_Generic:Conn_01x04
- removed J_BTN_R: BTN_R, Connector_JST:JST_XH_B4B-XH-A_1x04_P2.50mm_Vertical, symbol Connector_Generic:Conn_01x04
- removed J_BUZ: BUZ, Connector_JST:JST_XH_B2B-XH-A_1x02_P2.50mm_Vertical, symbol Connector_Generic:Conn_01x02
- removed J_HBAT: HELTEC_BAT, Connector_JST:JST_XH_B2B-XH-A_1x02_P2.50mm_Vertical, symbol Connector_Generic:Conn_01x02
- removed J_KEY: KEY, Connector_JST:JST_XH_B2B-XH-A_1x02_P2.50mm_Vertical, symbol Connector_Generic:Conn_01x02
- removed J_LCD: LCD, Connector_JST:JST_XH_B4B-XH-A_1x04_P2.50mm_Vertical, symbol Connector_Generic:Conn_01x04
- removed J_NFC: NFC, Connector_JST:JST_XH_B4B-XH-A_1x04_P2.50mm_Vertical, symbol Connector_Generic:Conn_01x04
- removed Q_BZ, Q_LB, Q_LR: AO3400A, Package_TO_SOT_SMD:SOT-23, symbol Transistor_FET:AO3400A
- removed Q_SCL, Q_SDA: BSS138, Package_TO_SOT_SMD:SOT-23, symbol Transistor_FET:BSS138
- removed R_GBZ, R_GLB, R_GLR, R_LLB: 100R, Resistor_SMD:R_0805_2012Metric_Pad1.20x1.40mm_HandSolder, symbol Device:R
- removed R_LLR: 150R, Resistor_SMD:R_0805_2012Metric_Pad1.20x1.40mm_HandSolder, symbol Device:R
- removed R_PDBZ, R_PDLB, R_PDLR: 100k, Resistor_SMD:R_0805_2012Metric_Pad1.20x1.40mm_HandSolder, symbol Device:R
- removed R_PUB, R_PUR: 10k, Resistor_SMD:R_0805_2012Metric_Pad1.20x1.40mm_HandSolder, symbol Device:R
- removed R_SB, R_SR: 1k, Resistor_SMD:R_0805_2012Metric_Pad1.20x1.40mm_HandSolder, symbol Device:R
- added C_BB1, C_BR1: 100nF, Capacitor_SMD:C_0805_2012Metric_Pad1.18x1.45mm_HandSolder, symbol Device:C
- added C_BULK1: 220uF 10V, Capacitor_THT:CP_Radial_D6.3mm_P2.50mm, symbol Device:C_Polarized
- added C_IN1: 22uF 10V, Capacitor_SMD:C_1206_3216Metric_Pad1.33x1.80mm_HandSolder, symbol Device:C
- added C_NFC1: 100uF 10V, Capacitor_THT:CP_Radial_D6.3mm_P2.50mm, symbol Device:C_Polarized
- added D_FLY1: 1N4148W, Diode_SMD:D_SOD-123, symbol Diode:1N4148W
- added J_BAT1: BAT, Connector_JST:JST_XH_B2B-XH-A_1x02_P2.50mm_Vertical, symbol Connector_Generic:Conn_01x02
- added J_BTN_B1: BTN_B, Connector_JST:JST_XH_B4B-XH-A_1x04_P2.50mm_Vertical, symbol Connector_Generic:Conn_01x04
- added J_BTN_R1: BTN_R, Connector_JST:JST_XH_B4B-XH-A_1x04_P2.50mm_Vertical, symbol Connector_Generic:Conn_01x04
- added J_BUZ1: BUZ, Connector_JST:JST_XH_B2B-XH-A_1x02_P2.50mm_Vertical, symbol Connector_Generic:Conn_01x02
- added J_HBAT1: HELTEC_BAT, Connector_JST:JST_XH_B2B-XH-A_1x02_P2.50mm_Vertical, symbol Connector_Generic:Conn_01x02
- added J_KEY1: KEY, Connector_JST:JST_XH_B2B-XH-A_1x02_P2.50mm_Vertical, symbol Connector_Generic:Conn_01x02
- added J_LCD1: LCD, Connector_JST:JST_XH_B4B-XH-A_1x04_P2.50mm_Vertical, symbol Connector_Generic:Conn_01x04
- added J_NFC1: NFC, Connector_JST:JST_XH_B4B-XH-A_1x04_P2.50mm_Vertical, symbol Connector_Generic:Conn_01x04
- added Q_BZ1, Q_LB1, Q_LR1: AO3400A, Package_TO_SOT_SMD:SOT-23, symbol Transistor_FET:AO3400A
- added Q_SCL1, Q_SDA1: BSS138, Package_TO_SOT_SMD:SOT-23, symbol Transistor_FET:BSS138
- added R_GBZ1, R_GLB1, R_GLR1, R_LLB1: 100R, Resistor_SMD:R_0805_2012Metric_Pad1.20x1.40mm_HandSolder, symbol Device:R
- added R_LLR1: 150R, Resistor_SMD:R_0805_2012Metric_Pad1.20x1.40mm_HandSolder, symbol Device:R
- added R_PDBZ1, R_PDLB1, R_PDLR1: 100k, Resistor_SMD:R_0805_2012Metric_Pad1.20x1.40mm_HandSolder, symbol Device:R
- added R_PUB1, R_PUR1: 10k, Resistor_SMD:R_0805_2012Metric_Pad1.20x1.40mm_HandSolder, symbol Device:R
- added R_SB1, R_SR1: 1k, Resistor_SMD:R_0805_2012Metric_Pad1.20x1.40mm_HandSolder, symbol Device:R
Connections:
- net +3V3: now also C_NFC1.1, J_NFC1.2 (Pin_2), Q_SCL1.1 (G), Q_SDA1.1 (G), R_PUB1.1, R_PUR1.1
- net +5V: now also D_FLY1.1 (K), J_BTN_B1.3 (Pin_3), J_BTN_R1.3 (Pin_3), J_BUZ1.1 (Pin_1), J_LCD1.2 (Pin_2)
- net BTN_B_IN: now also R_SB1.2
- net BTN_B_LEDK: now also J_BTN_B1.4 (Pin_4), R_LLB1.2
- net BTN_B_SW: now also C_BB1.1, J_BTN_B1.1 (Pin_1), R_PUB1.2, R_SB1.1
- net BTN_R_IN: now also R_SR1.2
- net BTN_R_LEDK: now also J_BTN_R1.4 (Pin_4), R_LLR1.2
- net BTN_R_SW: now also C_BR1.1, J_BTN_R1.1 (Pin_1), R_PUR1.2, R_SR1.1
- net BUZ_G: now also R_GBZ1.1
- net BUZ_K: now also D_FLY1.2 (A), J_BUZ1.2 (Pin_2), Q_BZ1.3 (D)
- net GND: now also C_BB1.2, C_BR1.2, C_BULK1.2, C_IN1.2, C_NFC1.2, J_BAT1.2 (Pin_2), J_BTN_B1.2 (Pin_2), J_BTN_R1.2 (Pin_2), J_HBAT1.2 (Pin_2), J_LCD1.1 (Pin_1), J_NFC1.1 (Pin_1), Q_BZ1.2 (S), Q_LB1.2 (S), Q_LR1.2 (S), R_PDBZ1.2, R_PDLB1.2, R_PDLR1.2
- net LED_B_G: now also R_GLB1.1
- net LED_B_K: now also Q_LB1.3 (D), R_LLB1.1
- net LED_R_G: now also R_GLR1.1
- net LED_R_K: now also Q_LR1.3 (D), R_LLR1.1
- net Q_BZ_G: now also Q_BZ1.1 (G), R_GBZ1.2, R_PDBZ1.1
- net Q_LB_G: now also Q_LB1.1 (G), R_GLB1.2, R_PDLB1.1
- net Q_LR_G: now also Q_LR1.1 (G), R_GLR1.2, R_PDLR1.1
- net SCL_3V3: now also J_NFC1.4 (Pin_4), Q_SCL1.2 (S)
- net SCL_5V: now also J_LCD1.4 (Pin_4), Q_SCL1.3 (D)
- net SDA_3V3: now also J_NFC1.3 (Pin_3), Q_SDA1.2 (S)
- net SDA_5V: now also J_LCD1.3 (Pin_3), Q_SDA1.3 (D)
- net VBAT_F: now also J_KEY1.1 (Pin_1)
- net VBAT_RAW: now also J_BAT1.1 (Pin_1)
- net VBAT_SW: now also C_BULK1.1, C_IN1.1, J_HBAT1.1 (Pin_1), J_KEY1.2 (Pin_2)
