File: hardware/carrier.kicad_sch (KiCad schematic)
At the start: 58 parts, among them J2 Heltec_J2, J3 Heltec_J3, U1 MT3608, U2 TCA9534PWR, U3 MAX98357A

Commit message: hardware: carrier schematic rebuilt as block-structured, A*-routed (replaces label-per-pin)
Other:
- note added: "Battery, key switch, 5 V boost"
- note added: "GPIO expander (0x20), button inputs"
- note added: "Heltec V4 headers"
- note added: "I2C level shifter, LCD (5 V), NFC (3.3 V)"
- note added: "I2S speaker amp"
- note added: "Low-side drivers: button LEDs, buzzer"
- note added: "Mounting holes"
- moved on the sheet: C_AMP1, C_AMP2, C_BB1, C_BR1, C_BULK1, C_BULK2, C_EXP1, C_IN1, C_NFC1, C_OUT1, C_OUT2, D1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
