File: hardware/carrier.kicad_pcb (KiCad board)
At the start: 2 copper layers, 90 x 60 mm, 62 parts, among them J2 Heltec_J2, J3 Heltec_J3, U1 MT3608, U2 TCA9534PWR, U3 NS4168, U4 XB8089D

Commit message: hardware: carrier takes power from the pack board (P5)
The cell protector, key switch, 5 V boost and their parts move to the pack
board; the carrier gets a 6-pin J_PWR1 (GND GND VBAT_SW +5V SDA_3V3 SCL_3V3).
The first block is now "Power in (from pack board)" and does not wire its
rails, so every rail pin gets its own power port.

make BOARD=carrier all is green (ERC, DRC parity, gerbers, jlc).

Co-Authored-By: Claude Opus 5.5 <noreply@anthropic.com>
Parts:
- removed C_IN1, C_OUT1, C_OUT2: 22uF 25V, Capacitor_SMD:C_1206_3216Metric_Pad1.33x1.80mm_HandSolder
- removed C_PROT1: 100nF, Capacitor_SMD:C_0805_2012Metric_Pad1.18x1.45mm_HandSolder
- removed D1: SS34, Diode_SMD:D_SMA
- removed F1: 2A PTC, Fuse:Fuse_1206_3216Metric_Pad1.42x1.75mm_HandSolder
- removed J_BAT1: BAT, Connector_JST:JST_XH_B4B-XH-A_1x04_P2.50mm_Vertical
- removed J_KEY1: KEY, Connector_JST:JST_XH_B4B-XH-A_1x04_P2.50mm_Vertical
- removed L1: 10uH 2A, Inductor_SMD:L_Bourns_SRN6045TA
- removed R_FB1: 75k, Resistor_SMD:R_0805_2012Metric_Pad1.20x1.40mm_HandSolder
- removed R_FB2: 10k, Resistor_SMD:R_0805_2012Metric_Pad1.20x1.40mm_HandSolder
- removed R_PROT1: 1k, Resistor_SMD:R_0805_2012Metric_Pad1.20x1.40mm_HandSolder
- removed U1: MT3608, Package_TO_SOT_SMD:SOT-23-6
- removed U4: XB8089D, Package_SO:SOIC-8-1EP_3.9x4.9mm_P1.27mm_EP2.41x3.3mm
- added J_PWR1: PWR, Connector_JST:JST_XH_B6B-XH-A_1x06_P2.50mm_Vertical, F.Cu at (13.0, 6.00)
Routing:
- net BTN_R_SW: track 203.5 -> 104.5 mm, vias 4 -> 3
- net BAT_N: track 64.9 -> 0.00 mm, vias 1 -> 0
- net SDA_3V3: track 79.0 -> 132.9 mm
- net VBAT_RAW: track 47.7 -> 0.00 mm, vias 1 -> 0
- net AMP_SD_R: track 71.8 -> 45.1 mm, vias 4 -> 2
- net +5V: track 185.0 -> 210.6 mm, vias 4 -> 1
- net GND: track 323.4 -> 299.4 mm, vias 8 -> 11
- net +3V3: track 135.6 -> 114.6 mm, vias 4 -> 6
- net BUZ_K: track 42.4 -> 23.1 mm, vias 1 -> 0
- net BTN_B_IN: track 47.9 -> 61.2 mm
- net SCL_3V3: track 85.2 -> 94.7 mm, vias 1 -> 0
- net PROT_VDD: track 9.17 -> 0.00 mm, vias 2 -> 0
- net SW: track 8.08 -> 0.00 mm
- net VBAT_F: track 6.75 -> 0.00 mm
- net I2S_DIN: track 79.0 -> 85.0 mm
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Other:
- board text added: "PACK GND GND BAT 5V SDA SCL"
- board text removed: "BAT + -"
- board text removed: "KEY"
