File: hardware/carrier.kicad_pcb (KiCad board)
At the start: 2 copper layers, 90 x 60 mm, 49 parts, among them J2 Heltec_J2, J3 Heltec_J3, U2 TCA9534PWR, U3 NS4168

Commit message: hardware: off-board 2-wire connectors back to XH-2
J_HBAT1, J_BUZ1 and J_SPK1 (carrier) and J_KEY1 (pack) go back to JST-XH B2B-XH-A (C158012) instead of 4-pin B4B-XH-A (C144395) with pins 3-4 left no-connect. XH_SPARE is gone from both boards; the freed width puts J_BTN_R1 back on the carrier's top edge. Regenerated: both boards ERC/DRC clean, 0 unrouted.
Parts:
- J_BUZ1, J_HBAT1, J_SPK1: footprint Connector_JST:JST_XH_B4B-XH-A_1x04_P2.50mm_Vertical -> Connector_JST:JST_XH_B2B-XH-A_1x02_P2.50mm_Vertical
- moved J_BTN_R1 60.8 mm to (41.0, 6.00), turned to 0 degrees
- moved J_HBAT1 8.50 mm to (30.5, 6.00)
- moved J_NFC1 4.00 mm to (72.0, 6.00)
- moved J_LCD1 3.00 mm to (56.5, 6.00)
- moved J_PWR1 3.00 mm to (10.0, 6.00)
Routing:
- net BTN_R_SW: track 104.5 -> 37.4 mm, vias 3 -> 0
- net +5V: track 210.6 -> 148.3 mm, vias 1 -> 3
- net +3V3: track 114.6 -> 150.3 mm, vias 6 -> 5
- net GND: track 299.4 -> 275.8 mm, vias 11 -> 13
- net SDA_3V3: track 132.9 -> 109.6 mm
- net LED_R_G: track 33.1 -> 44.1 mm, vias 0 -> 4
- net BUZ_G: track 51.0 -> 43.1 mm, vias 2 -> 4
- net BTN_B_IN: track 61.2 -> 54.0 mm, vias 2 -> 6
- net BTN_B_SW: track 30.3 -> 37.2 mm, vias 1 -> 0
- net SCL_5V: track 23.2 -> 30.0 mm, vias 2 -> 1
- net SPK_N: track 18.6 -> 14.1 mm
- net AMP_SD_R: track 45.1 -> 49.5 mm, vias 2 -> 4
- net BTN_R_IN: track 18.4 -> 22.5 mm
- net I2S_BCLK: track 76.9 -> 73.3 mm, vias 2 -> 0
- net I2S_LRCLK: track 83.9 -> 80.2 mm
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Other:
- board text added: "BTN_R SW GND L+ L-"
- board text removed: "BTN_R L- L+ GND SW"
