File: hardware/pack.kicad_sch (KiCad schematic)
At the start: 124 parts, among them U1 MT3608

Commit message: hardware: pack board routing and fab package (P4.2)
The QFN24/VQFN16 pads cannot take a 0.8 mm Power trunk, so the shunt
Kelvin sense now splits through an 0R into the INA3221 (plan P4.2), and the
two INA3221s sit in a cell's free middle band next to their shunts.
Freerouting: 7 passes, 0 unrouted; DRC --schematic-parity: 0 violations.
make BOARD=pack fab writes fab/pack/; make boards is green for both boards.

check_gerbers.py: NPTH_EXPECT / PTH_COMPONENT_MIN come from the board
module (the pack's holders and USB-C legitimately add drills).
gen_sch/gen_pcb: NOT_ASSEMBLED parts agree on in_bom; HIDE_REF.

Co-Authored-By: Claude Opus 5.5 <noreply@anthropic.com>
Parts:
- added R_SNSF1, R_SNSF2, R_SNSF3, R_SNSF4, R_SNSS1, R_SNSS2, R_SNSS3, R_SNSS4: 0R, Resistor_SMD:R_0805_2012Metric_Pad1.20x1.40mm_HandSolder, symbol Device:R
- BT1, BT2, BT3, BT4, TP_GND, TP_NRST, TP_SWCLK, TP_SWDIO: now left out of the parts list
Connections:
- net CELL1_F: now also R_SNSF1.1; no longer U_INA1.12 (IN+1)
- net CELL1_S: now also R_SNSS1.1; no longer U_INA1.11 (IN-1)
- net CELL2_F: now also R_SNSF2.1; no longer U_INA1.15 (IN+2)
- net CELL2_S: now also R_SNSS2.1; no longer U_INA1.14 (IN-2)
- net CELL3_F: now also R_SNSF3.1; no longer U_INA1.2 (IN+3)
- net CELL3_S: now also R_SNSS3.1; no longer U_INA1.1 (IN-3)
- net CELL4_F: now also R_SNSF4.1; no longer U_INA2.12 (IN+1)
- net CELL4_S: now also R_SNSS4.1; no longer U_INA2.1 (IN-3), U_INA2.11 (IN-1), U_INA2.14 (IN-2), U_INA2.15 (IN+2), U_INA2.2 (IN+3)
- new net INA_F1: R_SNSF1.2, U_INA1.12 (IN+1)
- new net INA_F2: R_SNSF2.2, U_INA1.15 (IN+2)
- new net INA_F3: R_SNSF3.2, U_INA1.2 (IN+3)
- new net INA_F4: R_SNSF4.2, U_INA2.12 (IN+1)
- new net INA_S1: R_SNSS1.2, U_INA1.11 (IN-1)
- new net INA_S2: R_SNSS2.2, U_INA1.14 (IN-2)
- new net INA_S3: R_SNSS3.2, U_INA1.1 (IN-3)
- new net INA_S4: R_SNSS4.2, U_INA2.1 (IN-3), U_INA2.11 (IN-1), U_INA2.14 (IN-2), U_INA2.15 (IN+2), U_INA2.2 (IN+3)

Commit message: hardware: pack board 96x90 with bottom-side MYOUNG holders
The Keystone 1042 holders were only 14.86 mm tall around an 18.3 mm
cell, so parts placed under them could not fit. Swap to MYOUNG
BH-18650-A6AJ012 (C19184084, THT, footprint in local.pretty from drawing
MY-CP-0373) on the bottom side, with the MF52 bead NTCs in the holder
floor window; every SMD part stays on top for single-side assembly. The
board shrinks from 140 x 100 to 96 x 90 mm.

gen_pcb.py: BOTTOM set flips footprints, project fp-lib-table adds the
local library. VPACK/SYS split from the BQ25601 pins through 1206 0R
jumpers so the rails can take the 0.8 mm Power class.

make boards is green (ERC, DRC parity, gerbers, jlc).

Co-Authored-By: Claude Opus 5.5 <noreply@anthropic.com>
Parts:
- added R_BAT1, R_BAT2, R_SYS1: 0R, Resistor_SMD:R_1206_3216Metric_Pad1.30x1.75mm_HandSolder, symbol Device:R
- BT1, BT2, BT3, BT4: footprint Battery:BatteryHolder_Keystone_1042_1x18650 -> local:BatteryHolder_MYOUNG_BH-18650-A6AJ012
- TH1, TH2, TH3, TH4: footprint Resistor_SMD:R_0805_2012Metric_Pad1.20x1.40mm_HandSolder -> local:NTC_Bead_P2.54mm; now left out of the parts list
Connections:
- net SYS: now also R_SYS1.2; no longer C_SYS.1, L_CHG.2, U_CHG.15 (SYS), U_CHG.16 (SYS)
- net VPACK: now also R_BAT1.2, R_BAT2.2; no longer C_BAT.1, U_CHG.13 (BAT), U_CHG.14 (BAT)
- new net BAT_CHG: C_BAT.1, R_BAT1.1, R_BAT2.1, U_CHG.13 (BAT), U_CHG.14 (BAT)
- new net SYS_CHG: C_SYS.1, L_CHG.2, R_SYS1.1, U_CHG.15 (SYS), U_CHG.16 (SYS)

Commit message: hardware: pack board without protector ICs, Basic diode-OR and TS pair
Cost cut after a ~$140 quote for 5 assembled boards (15 SMD Extended
types at ~$3 each). The per-cell MCU switches already default off, so a
dead or reset MCU leaves every cell open; with the 5 A fuses and the
BQ25601's CV/OVP they cover what the four XB8089D did. Holder- now goes
straight to GND. A single shared protector was rejected: with all
switches open the pack rail is 0 V and it would cut the MCU's ground
return, so the board could never boot.

- U_P1-4, R_PROT1-4, C_PROT1-4 removed.
- Diode-OR: 3x BAT54C -> 5x B5819W SOD-123 (C8598, Basic), one per
  cell in its own band and D_OR5 for SYS.
- TS bias 5.23k/30.9k -> 5.1k/30k (Basic): window 0/60 C -> 0.5/60.8 C.
- Sense taps 0R -> 10R: a reversed cell's crowbar now pulls the INA3221
  inputs below -0.3 V until the fuse clears; 10 Ohm limits the clamp
  current.
- power_budget.py drops the XB8089D current.

11 SMD Extended types (was 15), 105 placements (was 115).
make BOARD=pack all is green (ERC, DRC parity, gerbers, jlc).

Co-Authored-By: Claude Opus 5.5 <noreply@anthropic.com>
Parts:
- removed C_PROT1, C_PROT2, C_PROT3, C_PROT4: 100nF, Capacitor_SMD:C_0805_2012Metric_Pad1.18x1.45mm_HandSolder, symbol Device:C
- removed R_PROT1, R_PROT2, R_PROT3, R_PROT4: 1k, Resistor_SMD:R_0805_2012Metric_Pad1.20x1.40mm_HandSolder, symbol Device:R
- removed U_P1, U_P2, U_P3, U_P4: XB8089D, Package_SO:SOIC-8-1EP_3.9x4.9mm_P1.27mm_EP2.41x3.3mm, symbol local:XB8089D
- added D_OR4, D_OR5: B5819W, Diode_SMD:D_SOD-123, symbol Device:D_Schottky
- D_OR1, D_OR2, D_OR3: value BAT54C -> B5819W; footprint Package_TO_SOT_SMD:SOT-23 -> Diode_SMD:D_SOD-123; symbol Diode:BAT54C -> Device:D_Schottky
- RT1: value 5k23 -> 5k1
- RT2: value 30k9 -> 30k
- R_SNSF1, R_SNSF2, R_SNSF3, R_SNSF4, R_SNSS1, R_SNSS2, R_SNSS3, R_SNSS4: value 0R -> 10R
Connections:
- net CELL1_N is gone; now on net GND: BT1.2 (-), D_CB1.2 (A)
- net CELL2_N is gone; now on net GND: BT2.2 (-), D_CB2.2 (A)
- net CELL3_N is gone; now on net GND: BT3.2 (-), D_CB3.2 (A)
- net CELL4_N is gone; now on net GND: BT4.2 (-), D_CB4.2 (A)
- net CELL1_F: now also D_OR1.2 (A); no longer D_OR1.1
- net CELL2_F: now also D_OR2.2 (A); no longer D_OR1.2
- net CELL3_F: now also D_OR3.2 (A); no longer D_OR2.1
- net CELL4_F: now also D_OR4.2 (A); no longer D_OR2.2
- net SYS: now also D_OR5.2 (A); no longer D_OR3.1, D_OR3.2
- net VMCU_IN: now also D_OR1.1 (K), D_OR2.1 (K), D_OR3.1 (K), D_OR4.1 (K), D_OR5.1 (K); no longer D_OR1.3, D_OR2.3, D_OR3.3

Commit message: hardware: one PAC1934 replaces the two INA3221s on the pack board
Four channels in one chip (C623960, UQFN-16 4x4, KiCad
Sensor_Energy:PAC1934x-xJQ), cell n on channel n, with on-chip power
accumulators for coulomb counting. VBUS is read at SENSE+, which sits on
the fuse side of the shunt, so each channel still sees its own cell with
the switch open. ADDRSEL to GND = 0x10. SLOW/ALERT and PWRDN take the
two MCU pins the INA alerts used (28, 29), both pulled up so the monitor
runs without firmware; the pull-ups sit beside the MCU.

Shunt 20 -> 10 mOhm (FMF06FTHR010-LH, C105362, 1 W): the PAC1934 allows
only 500 mV across its sense pins, and with no protector IC a hard short
drives about 25 A per cell until the fuse clears. +-10 A full scale.

power_budget.py: monitor at its 5 uA SLEEP (PWRDN drops the
configuration), pack key-off 112 uA.

104 placements, 11 SMD Extended types; make BOARD=pack all is green.

Co-Authored-By: Claude Opus 5.5 <noreply@anthropic.com>
Parts:
- removed C_INA1, C_INA2: 100nF, Capacitor_SMD:C_0805_2012Metric_Pad1.18x1.45mm_HandSolder, symbol Device:C
- removed R_CRIT, R_WARN: 10k, Resistor_SMD:R_0805_2012Metric_Pad1.20x1.40mm_HandSolder, symbol Device:R
- removed U_INA1, U_INA2: INA3221, Package_DFN_QFN:Texas_RGV0016A_VQFN-16-1EP_4x4mm_P0.65mm_EP2.1x2.1mm, symbol Power_Management:INA3221
- added C_MON1, C_MON2: 100nF, Capacitor_SMD:C_0805_2012Metric_Pad1.18x1.45mm_HandSolder, symbol Device:C
- added R_ALERT, R_PWRDN: 10k, Resistor_SMD:R_0805_2012Metric_Pad1.20x1.40mm_HandSolder, symbol Device:R
- added U_MON: PAC1934T-I/JQ, Package_DFN_QFN:UQFN-16-1EP_4x4mm_P0.65mm_EP2.6x2.6mm, symbol Sensor_Energy:PAC1934x-xJQ
- R_SH1, R_SH2, R_SH3, R_SH4: value 20mOhm -> 10mOhm
Connections:
- net +3V3: now also C_MON1.1, C_MON2.1, R_ALERT.1, R_PWRDN.1, U_MON.15 (V_{DD}IO), U_MON.2 (V_{DD})
- net GND: now also C_MON1.2, C_MON2.2, U_MON.17 (EP), U_MON.3 (GND), U_MON.6 (ADDRSEL)
- net SCL_INT: now also U_MON.4 (SCL)
- net SDA_INT: now also U_MON.5 (SDA)
- net INA_CRIT renamed MON_ALERT
- net MON_ALERT: now also R_ALERT.2, U_MON.1 (SLOW)
- net INA_F1 renamed SNS_F1
- net SNS_F1: now also U_MON.11 (SENSE1+)
- net INA_F2 renamed SNS_F2
- net SNS_F2: now also U_MON.13 (SENSE2+)
- net INA_F3 renamed SNS_F3
- net SNS_F3: now also U_MON.8 (SENSE3+)
- net INA_F4 renamed SNS_F4
- net SNS_F4: now also U_MON.10 (SENSE4+)
- net INA_S1 renamed SNS_S1
- net SNS_S1: now also U_MON.12 (SENSE1-)
- net INA_S2 renamed SNS_S2
- net SNS_S2: now also U_MON.14 (SENSE2-)
- net INA_S3 renamed SNS_S3
- net SNS_S3: now also U_MON.7 (SENSE3-)
- net INA_S4 renamed SNS_S4
- net SNS_S4: now also U_MON.9 (SENSE4-)
- net INA_WARN renamed MON_PWRDN
- net MON_PWRDN: now also R_PWRDN.2, U_MON.16 (~{PWRDN})
- no-connect marks 18 -> 14
Other:
- note added: "Cell monitoring (PAC1934), diode-OR, 3V3 LDO"
- note removed: "Cell monitoring (INA3221 x2), diode-OR, 3V3 LDO"
