File: hardware/pack.kicad_sch (KiCad schematic)
At the start: 124 parts, among them U1 MT3608

Commit message: hardware: off-board 2-wire connectors back to XH-2
J_HBAT1, J_BUZ1 and J_SPK1 (carrier) and J_KEY1 (pack) go back to JST-XH B2B-XH-A (C158012) instead of 4-pin B4B-XH-A (C144395) with pins 3-4 left no-connect. XH_SPARE is gone from both boards; the freed width puts J_BTN_R1 back on the carrier's top edge. Regenerated: both boards ERC/DRC clean, 0 unrouted.
Parts:
- J_KEY1: footprint Connector_JST:JST_XH_B4B-XH-A_1x04_P2.50mm_Vertical -> Connector_JST:JST_XH_B2B-XH-A_1x02_P2.50mm_Vertical; symbol Connector_Generic:Conn_01x04 -> Connector_Generic:Conn_01x02
Connections:
- no-connect marks 14 -> 12
Changed lines of the file:
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@@
 	(wire
 		(pts
-			(xy 535.94 25.4)
-			(xy 574.04 25.4)
+			(xy 549.91 34.29)
+			(xy 574.04 34.29)
 		)
 		(stroke
@@
 	(wire
 		(pts
-			(xy 535.94 33.02)
-			(xy 541.02 33.02)
+			(xy 541.02 40.64)
+			(xy 549.91 40.64)
 		)
 		(stroke
@@
 	(wire
 		(pts
-			(xy 535.94 25.4)
-			(xy 535.94 33.02)
+			(xy 541.02 35.56)
+			(xy 541.02 40.64)
 		)
 		(stroke
@@
 	(wire
 		(pts
-			(xy 574.04 25.4)
-			(xy 574.04 34.29)
+			(xy 549.91 34.29)
+			(xy 549.91 40.64)
 		)
 		(stroke
@@
 	(wire
 		(pts
-			(xy 537.21 30.48)
-			(xy 541.02 30.48)
+			(xy 537.21 33.02)
+			(xy 541.02 33.02)
 		)
 		(stroke
@@
 	(wire
 		(pts
-			(xy 537.21 30.48)
+			(xy 537.21 33.02)
 			(xy 537.21 111.76)
 		)
@@
 	)
 	(no_connect
-		(at 541.02 35.56)
-	)
-	(no_connect
-		(at 541.02 38.1)
-	)
-	(no_connect
 		(at 596.9 58.42)
 	)
@@
 	(global_label "KEY_OUT"
 		(shape passive)
-		(at 537.21 25.4 0)
+		(at 551.18 34.29 0)
 		(fields_autoplaced yes)
 		(effects
@@
 	)
 	(symbol
-		(lib_id "Connector_Generic:Conn_01x04")
+		(lib_id "Connector_Generic:Conn_01x02")
 		(at 546.1 33.02 0)
 		(unit 1)
@@
 		(dnp no)
 		(property "Reference" "J_KEY1"
-			(at 546.1 27.94 0)
+			(at 546.1 30.48 0)
 			(effects
 				(font
@@
 		)
 		(property "Value" "KEY"
-			(at 546.1 40.64 0)
+			(at 546.1 38.1 0)
 			(effects
 				(font
@@
 			)
 		)
-		(property "Footprint" "Connector_JST:JST_XH_B4B-XH-A_1x04_P2.50mm_Vertical"
+		(property "Footprint" "Connector_JST:JST_XH_B2B-XH-A_1x02_P2.50mm_Vertical"
 			(at 546.1 33.02 0)
 			(effects
@@
 			)
 		)
-		(property "Description" "Generic connector, single row, 01x04, script generated (kicad-library-utils/schlib/autogen/connector/)"
+		(property "Description" "Generic connector, single row, 01x02, script generated (kicad-library-utils/schlib/autogen/connector/)"
 			(at 546.1 33.02 0)
 			(effects
@@
 		(pin "2"
 		)
-		(pin "3"
-		)
-		(pin "4"
-		)
 		(instances
