File: hardware/lipo.kicad_sch (KiCad schematic)
At the start: 59 parts

Commit message: hardware: LiPo board Extended types 7 -> 4
AO3407A -> AO3401A (Basic) with a 10 V MMSZ5240B (Preferred) gate clamp
under its 12 V VGS limit; SMBJ15A moves to the Preferred C19077569.
Checked against the live JLCPCB Basic/Preferred catalog.

Co-Authored-By: Claude Opus 5.5 <noreply@anthropic.com>
Parts:
- D_GZ1: value BZT52C12 -> MMSZ5240B
- Q_REV1: value AO3407A -> AO3401A
Changed lines of the file:
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@@
 			)
 		)
-		(property "Value" "AO3407A"
+		(property "Value" "AO3401A"
 			(at 76.2 43.18 0)
 			(effects
@@
 			)
 		)
-		(property "Value" "BZT52C12"
+		(property "Value" "MMSZ5240B"
 			(at 88.9 60.96 0)
 			(effects
