File: hardware/pack_b.kicad_sch (KiCad schematic)
At the start: 114 parts, among them U1 MT3608

Commit message: hardware: pack charger NTC hand-soldered, drops its Extended fee
TH_CHG (0805 10k B3435) leaves the JLC BOM/CPL on both pack variants; no
Basic/Preferred NTC exists. Left off, TS reads cold and charging stays
off. ORDERING.md: pack fees 11 -> 10, LiPo fees 7 -> 4, MT3608 ->
TPS61040 rejected (~89 mA worst case vs 82 mA peak +5V load).

Co-Authored-By: Claude Opus 5.5 <noreply@anthropic.com>
Parts:
- TH_CHG: now left out of the parts list
Changed lines of the file:
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@@
 		(unit 1)
 		(exclude_from_sim no)
-		(in_bom yes)
+		(in_bom no)
 		(on_board yes)
 		(dnp no)
