File: hardware/lipo_tme.kicad_pcb (KiCad board)
At the start: 2 copper layers, 70 x 50 mm, 62 parts

Commit message: hw: TME substitutes for parts TME lacks or sells only by the reel
Checked on tme.eu 2026-10-02 (inventoryLevel, minimum, multiple):
- INA228AIDGSR (no stock, every variant) -> INA226AIDGSR, same VSSOP-10
  pins and A1/A0 addresses; 0.5 uA shutdown in the power model.
- LiPo TPS54302DDCR (no stock) -> TPS563200DDCR, same SOT-23-6 pins;
  VFB 0.765 V so R_FBA1 22k (4.07 V) and R_FBB1 56k (5.05 V), L 3.3 uH
  per TI's 2.2-4.7 uH table. VIN is 17 V max (19 V abs): 3S only.
- SRN6045TA-100M (not at TME), SRN60454R7Y-BOU-0 (1000 minimum) ->
  SRN6045-3R3Y on the same pads (MCP1640 takes 2.2-10 uH).
- SF-1206F500-2 (5000 reel) -> Bel C1F-5, 5 A fast 1206, I2t 0.83 A2s.
- SS34-YAN (no stock) -> SSA34-E3/61T, SMA (TME's SS34s are SMC).
- CL21B105KBFNNNE (no stock) -> CL21B105KAFNNNE 25 V (all on <= 5 V).
- PCM5100APWR (70 tube / 2000 reel only) leaves the TME list: LCSC/Mouser.

tme_all.py rounds to TME's minimum as well as its multiple (C1F-5: 5).
lipo_tme and pack_tme regenerated: ERC/DRC 0, gerbers ok.

Co-Authored-By: Claude Opus 5.5 <noreply@anthropic.com>
Parts:
- L_A, L_B: value 10uH 2A -> 3u3
- R_FBA1: value 30k -> 22k
- R_FBB1: value 75k -> 56k
- U_BA, U_BB: value TPS54302DDCR -> TPS563200DDCR
Changed lines of the file:
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@@
 			)
 		)
-		(property "Value" "30k"
+		(property "Value" "22k"
 			(at 0 1.65 0)
 			(layer "F.Fab")
@@
 			)
 		)
-		(property "Value" "75k"
+		(property "Value" "56k"
 			(at 0 1.65 0)
 			(layer "F.Fab")
@@
 			)
 		)
-		(property "Value" "TPS54302DDCR"
+		(property "Value" "TPS563200DDCR"
 			(at 0 2.4 0)
 			(layer "F.Fab")
@@
 			)
 		)
-		(property "Value" "10uH 2A"
+		(property "Value" "3u3"
 			(at 0 4.2 0)
 			(layer "F.Fab")
@@
 			)
 		)
-		(property "Value" "TPS54302DDCR"
+		(property "Value" "TPS563200DDCR"
 			(at 0 2.4 0)
 			(layer "F.Fab")
@@
 			)
 		)
-		(property "Value" "10uH 2A"
+		(property "Value" "3u3"
 			(at 0 4.2 0)
 			(layer "F.Fab")
