File: hardware/lipo_tme.kicad_sch (KiCad schematic)
At the start: 62 parts

Commit message: hw: TME substitutes for parts TME lacks or sells only by the reel
Checked on tme.eu 2026-10-02 (inventoryLevel, minimum, multiple):
- INA228AIDGSR (no stock, every variant) -> INA226AIDGSR, same VSSOP-10
  pins and A1/A0 addresses; 0.5 uA shutdown in the power model.
- LiPo TPS54302DDCR (no stock) -> TPS563200DDCR, same SOT-23-6 pins;
  VFB 0.765 V so R_FBA1 22k (4.07 V) and R_FBB1 56k (5.05 V), L 3.3 uH
  per TI's 2.2-4.7 uH table. VIN is 17 V max (19 V abs): 3S only.
- SRN6045TA-100M (not at TME), SRN60454R7Y-BOU-0 (1000 minimum) ->
  SRN6045-3R3Y on the same pads (MCP1640 takes 2.2-10 uH).
- SF-1206F500-2 (5000 reel) -> Bel C1F-5, 5 A fast 1206, I2t 0.83 A2s.
- SS34-YAN (no stock) -> SSA34-E3/61T, SMA (TME's SS34s are SMC).
- CL21B105KBFNNNE (no stock) -> CL21B105KAFNNNE 25 V (all on <= 5 V).
- PCM5100APWR (70 tube / 2000 reel only) leaves the TME list: LCSC/Mouser.

tme_all.py rounds to TME's minimum as well as its multiple (C1F-5: 5).
lipo_tme and pack_tme regenerated: ERC/DRC 0, gerbers ok.

Co-Authored-By: Claude Opus 5.5 <noreply@anthropic.com>
Parts:
- L_A, L_B: value 10uH 2A -> 3u3
- R_FBA1: value 30k -> 22k
- R_FBB1: value 75k -> 56k
- U_BA, U_BB: value TPS54302DDCR -> TPS563200DDCR; symbol Regulator_Switching:TPS54302 -> Regulator_Switching:TPS563200
Changed lines of the file:
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@@
 	(wire
 		(pts
-			(xy 193.04 40.64)
-			(xy 198.12 40.64)
+			(xy 193.04 43.18)
+			(xy 198.12 43.18)
 		)
 		(stroke
@@
 		(pts
 			(xy 198.12 29.21)
-			(xy 198.12 40.64)
+			(xy 198.12 43.18)
 		)
 		(stroke
@@
 	(wire
 		(pts
-			(xy 193.04 101.6)
-			(xy 198.12 101.6)
+			(xy 193.04 104.14)
+			(xy 198.12 104.14)
 		)
 		(stroke
@@
 		(pts
 			(xy 198.12 90.17)
-			(xy 198.12 101.6)
+			(xy 198.12 104.14)
 		)
 		(stroke
@@
 	(wire
 		(pts
-			(xy 193.04 43.18)
-			(xy 208.28 43.18)
+			(xy 193.04 40.64)
+			(xy 208.28 40.64)
 		)
 		(stroke
@@
 		(pts
 			(xy 208.28 36.83)
-			(xy 208.28 43.18)
+			(xy 208.28 40.64)
 		)
 		(stroke
@@
 	(wire
 		(pts
-			(xy 193.04 104.14)
-			(xy 208.28 104.14)
+			(xy 193.04 101.6)
+			(xy 208.28 101.6)
 		)
 		(stroke
@@
 		(pts
 			(xy 208.28 97.79)
-			(xy 208.28 104.14)
+			(xy 208.28 101.6)
 		)
 		(stroke
@@
 	)
 	(symbol
-		(lib_id "Regulator_Switching:TPS54302")
+		(lib_id "Regulator_Switching:TPS563200")
 		(at 182.88 43.18 0)
 		(unit 1)
@@
 			)
 		)
-		(property "Value" "TPS54302DDCR"
-			(at 182.88 36.83 0)
+		(property "Value" "TPS563200DDCR"
+			(at 180.34 36.83 0)
 			(effects
 				(font
@@
 		)
 		(property "Footprint" "Package_TO_SOT_SMD:TSOT-23-6"
-			(at 184.15 52.07 0)
+			(at 184.15 49.53 0)
 			(effects
 				(font
@@
 			)
 		)
-		(property "Datasheet" "http://www.ti.com/lit/ds/symlink/tps54302.pdf"
-			(at 175.26 34.29 0)
+		(property "Datasheet" "http://www.ti.com/lit/ds/symlink/tps563200.pdf"
+			(at 182.88 43.18 0)
 			(effects
 				(font
@@
 			)
 		)
-		(property "Description" "3A, 4.5 to 28V Input, EMI Friendly integrated switch synchronous step-down regulator, pulse-skipping, SOT-23-6"
+		(property "Description" "3A Synchronous Step-Down Voltage Regulator, Adjustable Output Voltage, 4.5-17V Input Voltage, SOT-23-6"
 			(at 182.88 43.18 0)
 			(effects
@@
 		(pin "1"
 		)
-		(pin "6"
-		)
 		(pin "2"
 		)
+		(pin "6"
+		)
 		(pin "4"
 		)
@@
 			)
 		)
-		(property "Value" "10uH 2A"
+		(property "Value" "3u3"
 			(at 230.505 40.64 90)
 			(effects
@@
 			)
 		)
-		(property "Value" "30k"
+		(property "Value" "22k"
 			(at 248.92 50.8 90)
 			(effects
@@
 	)
 	(symbol
-		(lib_id "Regulator_Switching:TPS54302")
+		(lib_id "Regulator_Switching:TPS563200")
 		(at 182.88 104.14 0)
 		(unit 1)
@@
 			)
 		)
-		(property "Value" "TPS54302DDCR"
-			(at 182.88 97.79 0)
+		(property "Value" "TPS563200DDCR"
+			(at 180.34 97.79 0)
 			(effects
 				(font
@@
 		)
 		(property "Footprint" "Package_TO_SOT_SMD:TSOT-23-6"
-			(at 184.15 113.03 0)
+			(at 184.15 110.49 0)
 			(effects
 				(font
@@
 			)
 		)
-		(property "Datasheet" "http://www.ti.com/lit/ds/symlink/tps54302.pdf"
-			(at 175.26 95.25 0)
+		(property "Datasheet" "http://www.ti.com/lit/ds/symlink/tps563200.pdf"
+			(at 182.88 104.14 0)
 			(effects
 				(font
@@
 			)
 		)
-		(property "Description" "3A, 4.5 to 28V Input, EMI Friendly integrated switch synchronous step-down regulator, pulse-skipping, SOT-23-6"
+		(property "Description" "3A Synchronous Step-Down Voltage Regulator, Adjustable Output Voltage, 4.5-17V Input Voltage, SOT-23-6"
 			(at 182.88 104.14 0)
 			(effects
@@
 		(pin "1"
 		)
-		(pin "6"
-		)
 		(pin "2"
 		)
+		(pin "6"
+		)
 		(pin "4"
 		)
@@
 			)
 		)
-		(property "Value" "10uH 2A"
+		(property "Value" "3u3"
 			(at 230.505 101.6 90)
 			(effects
@@
 			)
 		)
-		(property "Value" "75k"
+		(property "Value" "56k"
 			(at 248.92 111.76 90)
 			(effects
