File: hardware/pack_tme.kicad_sch (KiCad schematic)
At the start: 129 parts, among them U1 MCP1640T-I/CHY

Commit message: hw: pack TME schematic titles the MCU block STM32L072
Co-Authored-By: Claude Opus 5.5 <noreply@anthropic.com>
Other:
- note added: "STM32L072 MCU, reset/boot, test pads"
- note removed: "STM32C071 MCU, reset/boot, test pads"
Changed lines of the file:
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@@
 		)
 	)
-	(text "STM32C071 MCU, reset/boot, test pads"
+	(text "STM32L072 MCU, reset/boot, test pads"
 		(exclude_from_sim no)
 		(at 383.54 17.78 0)

Commit message: hw: TME substitutes for parts TME lacks or sells only by the reel
Checked on tme.eu 2026-10-02 (inventoryLevel, minimum, multiple):
- INA228AIDGSR (no stock, every variant) -> INA226AIDGSR, same VSSOP-10
  pins and A1/A0 addresses; 0.5 uA shutdown in the power model.
- LiPo TPS54302DDCR (no stock) -> TPS563200DDCR, same SOT-23-6 pins;
  VFB 0.765 V so R_FBA1 22k (4.07 V) and R_FBB1 56k (5.05 V), L 3.3 uH
  per TI's 2.2-4.7 uH table. VIN is 17 V max (19 V abs): 3S only.
- SRN6045TA-100M (not at TME), SRN60454R7Y-BOU-0 (1000 minimum) ->
  SRN6045-3R3Y on the same pads (MCP1640 takes 2.2-10 uH).
- SF-1206F500-2 (5000 reel) -> Bel C1F-5, 5 A fast 1206, I2t 0.83 A2s.
- SS34-YAN (no stock) -> SSA34-E3/61T, SMA (TME's SS34s are SMC).
- CL21B105KBFNNNE (no stock) -> CL21B105KAFNNNE 25 V (all on <= 5 V).
- PCM5100APWR (70 tube / 2000 reel only) leaves the TME list: LCSC/Mouser.

tme_all.py rounds to TME's minimum as well as its multiple (C1F-5: 5).
lipo_tme and pack_tme regenerated: ERC/DRC 0, gerbers ok.

Co-Authored-By: Claude Opus 5.5 <noreply@anthropic.com>
Parts:
- L1: value 4u7 2A -> 3u3
- U_MON1, U_MON2, U_MON3, U_MON4: value INA228AIDGSR -> INA226AIDGSR; symbol Sensor_Energy:INA228 -> Sensor_Energy:INA226
Other:
- note added: "Cell 1 branch + INA226"
- note added: "Cell 2 branch + INA226"
- note added: "Cell 3 branch + INA226"
- note added: "Cell 4 branch + INA226"
- note removed: "Cell 1 branch + INA228"
- note removed: "Cell 2 branch + INA228"
- note removed: "Cell 3 branch + INA228"
- note removed: "Cell 4 branch + INA228"
Changed lines of the file:
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@@
 		)
 	)
-	(text "Cell 1 branch + INA228"
+	(text "Cell 1 branch + INA226"
 		(exclude_from_sim no)
 		(at 15.24 195.58 0)
@@
 		)
 	)
-	(text "Cell 2 branch + INA228"
+	(text "Cell 2 branch + INA226"
 		(exclude_from_sim no)
 		(at 116.84 195.58 0)
@@
 		)
 	)
-	(text "Cell 3 branch + INA228"
+	(text "Cell 3 branch + INA226"
 		(exclude_from_sim no)
 		(at 218.44 195.58 0)
@@
 		)
 	)
-	(text "Cell 4 branch + INA228"
+	(text "Cell 4 branch + INA226"
 		(exclude_from_sim no)
 		(at 320.04 195.58 0)
@@
 			)
 		)
-		(property "Value" "4u7 2A"
+		(property "Value" "3u3"
 			(at 619.125 43.18 90)
 			(effects
@@
 	)
 	(symbol
-		(lib_id "Sensor_Energy:INA228")
+		(lib_id "Sensor_Energy:INA226")
 		(at 76.2 261.62 0)
 		(unit 1)
@@
 			)
 		)
-		(property "Value" "INA228AIDGSR"
+		(property "Value" "INA226AIDGSR"
 			(at 80.01 250.19 0)
 			(effects
@@
 			)
 		)
-		(property "Datasheet" "https://www.ti.com/lit/ds/symlink/ina228.pdf"
+		(property "Datasheet" "http://www.ti.com/lit/ds/symlink/ina226.pdf"
 			(at 85.09 264.16 0)
 			(effects
@@
 			)
 		)
-		(property "Description" "High-Side or Low-Side Measurement, Bi-Directional Current and Power Monitor (0-85V) with I2C, SMBus-, and PMBus-Compatible Interface, VSSOP-10"
+		(property "Description" "High-Side or Low-Side Measurement, Bi-Directional Current and Power Monitor (0-36V) with I2C Compatible Interface, VSSOP-10"
 			(at 76.2 261.62 0)
 			(effects
@@
 	)
 	(symbol
-		(lib_id "Sensor_Energy:INA228")
+		(lib_id "Sensor_Energy:INA226")
 		(at 177.8 261.62 0)
 		(unit 1)
@@
 			)
 		)
-		(property "Value" "INA228AIDGSR"
+		(property "Value" "INA226AIDGSR"
 			(at 181.61 250.19 0)
 			(effects
@@
 			)
 		)
-		(property "Datasheet" "https://www.ti.com/lit/ds/symlink/ina228.pdf"
+		(property "Datasheet" "http://www.ti.com/lit/ds/symlink/ina226.pdf"
 			(at 186.69 264.16 0)
 			(effects
@@
 			)
 		)
-		(property "Description" "High-Side or Low-Side Measurement, Bi-Directional Current and Power Monitor (0-85V) with I2C, SMBus-, and PMBus-Compatible Interface, VSSOP-10"
+		(property "Description" "High-Side or Low-Side Measurement, Bi-Directional Current and Power Monitor (0-36V) with I2C Compatible Interface, VSSOP-10"
 			(at 177.8 261.62 0)
 			(effects
@@
 	)
 	(symbol
-		(lib_id "Sensor_Energy:INA228")
+		(lib_id "Sensor_Energy:INA226")
 		(at 279.4 261.62 0)
 		(unit 1)
@@
 			)
 		)
-		(property "Value" "INA228AIDGSR"
+		(property "Value" "INA226AIDGSR"
 			(at 283.21 250.19 0)
 			(effects
@@
 			)
 		)
-		(property "Datasheet" "https://www.ti.com/lit/ds/symlink/ina228.pdf"
+		(property "Datasheet" "http://www.ti.com/lit/ds/symlink/ina226.pdf"
 			(at 288.29 264.16 0)
 			(effects
@@
 			)
 		)
-		(property "Description" "High-Side or Low-Side Measurement, Bi-Directional Current and Power Monitor (0-85V) with I2C, SMBus-, and PMBus-Compatible Interface, VSSOP-10"
+		(property "Description" "High-Side or Low-Side Measurement, Bi-Directional Current and Power Monitor (0-36V) with I2C Compatible Interface, VSSOP-10"
 			(at 279.4 261.62 0)
 			(effects
@@
 	)
 	(symbol
-		(lib_id "Sensor_Energy:INA228")
+		(lib_id "Sensor_Energy:INA226")
 		(at 381 261.62 0)
 		(unit 1)
@@
 			)
 		)
-		(property "Value" "INA228AIDGSR"
+		(property "Value" "INA226AIDGSR"
 			(at 384.81 250.19 0)
 			(effects
@@
 			)
 		)
-		(property "Datasheet" "https://www.ti.com/lit/ds/symlink/ina228.pdf"
+		(property "Datasheet" "http://www.ti.com/lit/ds/symlink/ina226.pdf"
 			(at 389.89 264.16 0)
 			(effects
@@
 			)
 		)
-		(property "Description" "High-Side or Low-Side Measurement, Bi-Directional Current and Power Monitor (0-85V) with I2C, SMBus-, and PMBus-Compatible Interface, VSSOP-10"
+		(property "Description" "High-Side or Low-Side Measurement, Bi-Directional Current and Power Monitor (0-36V) with I2C Compatible Interface, VSSOP-10"
 			(at 381 261.62 0)
 			(effects
