File: hardware/kicad/carrier.kicad_pcb (KiCad board)
At the start: 2 copper layers, 90 x 60 mm, 49 parts, among them J2 Heltec_J2, J3 Heltec_J3, U2 TCA9534PWR, U3 NS4168

Commit message: hardware: UART debug header on all boards, I2C header and rail test pads on carrier, SDA/SCL pads on pack
Header is 1x3 2.54 mm (GND, MCU TX, MCU RX), hand-soldered, kept out of the BOM.
Carrier uses Heltec UART0 (GPIO43/44), STM32 boards USART1 (PA9/PA10).

Co-Authored-By: Claude Sonnet 5.5 <noreply@anthropic.com>
Parts:
- added J_I2C1: I2C, Connector_PinHeader_2.54mm:PinHeader_1x04_P2.54mm_Vertical, F.Cu at (56.0, 55.5)
- added J_UART1: UART, Connector_PinHeader_2.54mm:PinHeader_1x03_P2.54mm_Vertical, F.Cu at (47.0, 55.5)
- added TP_3V3: 3V3, TestPoint:TestPoint_Pad_D1.5mm, F.Cu at (68.0, 55.5)
- added TP_5V: 5V, TestPoint:TestPoint_Pad_D1.5mm, F.Cu at (70.5, 55.5)
- added TP_GND: GND, TestPoint:TestPoint_Pad_D1.5mm, F.Cu at (75.5, 55.5)
- added TP_VSW: VBAT_SW, TestPoint:TestPoint_Pad_D1.5mm, F.Cu at (73.0, 55.5)
Connections:
- J2 pad 5: unconnected-(J2-Pin_5-Pad5) -> UART_RX
- J2 pad 6: unconnected-(J2-Pin_6-Pad6) -> UART_TX
Routing:
- net SCL_3V3: track 93.3 -> 180.9 mm, vias 2 -> 3
- net VBAT_SW: track 62.8 -> 140.4 mm
- net GND: track 275.8 -> 345.7 mm, vias 13 -> 8
- net +5V: track 148.3 -> 217.1 mm, vias 3 -> 1
- net SDA_3V3: track 109.6 -> 163.4 mm, vias 2 -> 3
- net +3V3: track 150.3 -> 190.8 mm, vias 5 -> 2
- net UART_TX: track 0.00 -> 12.4 mm
- net I2S_DIN: track 82.5 -> 93.1 mm, vias 0 -> 2
- net LED_R_G: track 44.1 -> 33.7 mm, vias 4 -> 0
- net BTN_B_IN: track 54.0 -> 63.9 mm, vias 6 -> 2
- net I2S_BCLK: track 73.3 -> 81.1 mm, vias 0 -> 2
- net BTN_B_SW: track 37.2 -> 30.3 mm, vias 0 -> 1
- net UART_RX: track 0.00 -> 6.84 mm
- net BTN_R_IN: track 22.5 -> 16.1 mm
- net Q_BZ_G: track 5.58 -> 10.0 mm
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Other:
- board text added: "3V3"
- board text added: "5V"
- board text added: "GND"
- board text added: "I2C GND 3V3 SDA SCL"
- board text added: "UART GND TX RX"
- board text added: "VSW"

Commit message: hardware: KiCad 10 pipeline fixes, +5V reservoir caps, NS4168 1uF, pack UART header off the holders
KiCad 9 -> 10.0.7 broke the generators even on HEAD:
- gen_sch: libraries moved (hide yes) from effects to the property; read both,
  write it back into effects (KiCad 9 format), so hidden fields stop showing
  on every sheet and stop blocking the schematic router. Add the title block.
- gen_pcb: SetDoNotAllowCopperPour -> SetDoNotAllowZoneFills; copy the symbol's
  Datasheet/Description/Sim fields onto footprints (schematic parity now fails
  DRC); refuse THT pads under bottom-side parts (PTH_UNDER_OK allowlist).
- route.py: Power class routed at +40 um (Freerouting's octagons undercut 0.8 mm
  round ends, KiCad 10 exports no clearance margin), falling back to no margin
  if that leaves a connection unrouted; strip dangling stubs after SES import.
- pack: USB-C shield pin S1 -> SH; pack_tme: VSSOP-10 -> MSOP-10 footprint.

Design changes from the Konnect MCP review and datasheet check:
- carrier: C_5V1 10 uF + C_5V2 100 nF on +5V at J_PWR1 (no local cap before);
  C_AMP2 100 nF -> 1 uF per NS4168 datasheet (100 uF || 1 uF). carrier_tme
  places the new caps clear of its DAC.
- pack/pack_tme: J_UART1 sat under BT4 (bottom-side 18650 holder), caught by
  KiCad 10's pth_inside_courtyard; moved to the right strip, label in pin order.
  The NTC beads stay in the holder window (check ignored, gen_pcb enforces it).
- Docs: ORDERING counts, NS4168/TCA9534/BSS138/1N4148W datasheet check,
  TCA9534 P6/P7 firmware note.

All six boards: ERC 0, DRC 0 (0 unconnected, 0 parity), gerbers ok.

Co-Authored-By: Claude Opus 5.5 <noreply@anthropic.com>
Parts:
- added C_5V1: 10uF, Capacitor_SMD:C_0805_2012Metric_Pad1.18x1.45mm_HandSolder, F.Cu at (25.0, 14.5)
- added C_5V2: 100nF, Capacitor_SMD:C_0805_2012Metric_Pad1.18x1.45mm_HandSolder, F.Cu at (29.5, 14.5)
- C_AMP2: value 100nF -> 1uF
Routing:
- net GND: track 345.7 -> 322.7 mm, vias 8 -> 9
- net SCL_3V3: track 180.9 -> 192.1 mm, vias 3 -> 2
- net LED_B_G: track 48.2 -> 59.3 mm
- net VBAT_SW: track 140.4 -> 149.2 mm
- net I2S_LRCLK: track 83.5 -> 90.9 mm, vias 1 -> 2
- net SCL_5V: track 33.6 -> 28.6 mm, vias 1 -> 2
- net AMP_SD_R: track 51.5 -> 47.0 mm, vias 4 -> 0
- net Q_BZ_G: track 10.0 -> 5.58 mm
- net SDA_3V3: track 163.4 -> 167.8 mm, vias 3 -> 4
- net BTN_R_LEDK: track 44.4 -> 47.7 mm
- net +5V: track 217.1 -> 220.1 mm, vias 1 -> 4
- net BTN_R_SW: track 37.6 -> 40.5 mm, vias 0 -> 1
- net BTN_B_IN: track 63.9 -> 61.1 mm, vias 2 -> 4
- net SDA_5V: track 37.7 -> 35.3 mm
- net I2S_DIN: track 93.1 -> 95.4 mm
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