File: hardware/kicad/carrier.kicad_pcb (KiCad board)
At the start: 2 copper layers, 90 x 60 mm, 57 parts, among them J2 Heltec_J2, J3 Heltec_J3, U2 TCA9534PWR, U3 NS4168

Commit message: hardware: 3.5" ILI9488 SPI TFT replaces the Newhaven LCD
Carrier and carrier_tme: J_LCD1 XH-8 (VCC GND CS RST DC MOSI SCK LED,
the module header order; CS tied low). SPI3 on GPIO43/44, PWM backlight
on GPIO6 (R_BLPD1), DC/RST on TCA9534 P6/P7, buttons polled. The P4/P5
native-pin option was dropped: the Heltec GNSS receptacle opens toward
those pins. Removed the I2C level shifter, R_INT1/EXP_INT and J_UART1;
J_NFC1 moved to the bottom edge. Both boards: 0 unrouted, ERC/DRC/parity 0.

Lid rebuilt from the LCDWiki MSP3520 drawing: 98 x 56.34, M3 bosses on
92 x 49.5 (r3.0, 4.5 high), 80 x 51 viewing window, 11.5 mm depth.
make mech green. Power model: backlight duty is now the mean PWM level.

Co-Authored-By: Claude Opus 5.5 <noreply@anthropic.com>
Parts:
- removed J_UART1: UART, Connector_PinHeader_2.54mm:PinHeader_1x03_P2.54mm_Vertical
- removed Q_SCL1, Q_SDA1: BSS138, Package_TO_SOT_SMD:SOT-23
- removed R_INT1: 10k, Resistor_SMD:R_0805_2012Metric_Pad1.20x1.40mm_HandSolder
- removed R_SCL5, R_SDA5: 4k7, Resistor_SMD:R_0805_2012Metric_Pad1.20x1.40mm_HandSolder
- added R_BLPD1: 10k, Resistor_SMD:R_0805_2012Metric_Pad1.20x1.40mm_HandSolder, F.Cu at (66.0, 22.8)
- J_LCD1: footprint Connector_JST:JST_XH_B4B-XH-A_1x04_P2.50mm_Vertical -> Connector_JST:JST_XH_B8B-XH-A_1x08_P2.50mm_Vertical
- moved J_NFC1 53.9 mm to (51.0, 55.6), turned to 180 degrees
Connections:
- J2 pad 5: UART_RX -> LCD_MOSI
- J2 pad 6: UART_TX -> LCD_SCK
- J3 pad 17: EXP_INT -> LCD_BL
- J_LCD1 pad 1: GND -> +5V
- J_LCD1 pad 2: +5V -> GND
- J_LCD1 pad 3: SDA_5V -> GND
- J_LCD1 pad 4: SCL_5V -> LCD_RST
- U2 pad 11: unconnected-(U2-P6-Pad11) -> LCD_DC
- U2 pad 12: unconnected-(U2-P7-Pad12) -> LCD_RST
- U2 pad 13: EXP_INT -> unconnected-(U2-~{INT}-Pad13)
Routing:
- net LCD_SCK: track 0.00 -> 87.2 mm, vias 0 -> 1
- net LCD_MOSI: track 0.00 -> 73.6 mm
- net SCL_3V3: track 192.1 -> 137.0 mm, vias 2 -> 3
- net LCD_BL: track 0.00 -> 48.6 mm
- net SDA_5V: track 35.3 -> 0.00 mm, vias 2 -> 0
- net BUZ_G: track 42.6 -> 75.6 mm
- net SCL_5V: track 28.6 -> 0.00 mm, vias 2 -> 0
- net EXP_INT: track 26.5 -> 0.00 mm
- net +3V3: track 189.4 -> 163.2 mm, vias 2 -> 1
- net +5V: track 220.1 -> 194.2 mm, vias 4 -> 2
- net LCD_DC: track 0.00 -> 20.0 mm, vias 0 -> 2
- net LCD_RST: track 0.00 -> 17.8 mm, vias 0 -> 2
- net I2S_DIN: track 95.4 -> 80.7 mm
- net LED_B_G: track 59.3 -> 45.0 mm
- net BTN_B_SW: track 28.3 -> 41.0 mm, vias 1 -> 0
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Other:
- board text added: "LCD 5V GND CS0 RST DC MOSI SCK BL"
- board text added: "NFC SCL SDA 3V3 GND"
- board text removed: "LCD GND 5V SDA SCL"
- board text removed: "NFC GND 3V3 SDA SCL"
- board text removed: "UART GND TX RX"
