File: hardware/kicad/pack.kicad_pcb (KiCad board)
At the start: 2 copper layers, 96 x 90 mm, 124 parts, among them U1 MT3608

Commit message: hardware: UART debug header on all boards, I2C header and rail test pads on carrier, SDA/SCL pads on pack
Header is 1x3 2.54 mm (GND, MCU TX, MCU RX), hand-soldered, kept out of the BOM.
Carrier uses Heltec UART0 (GPIO43/44), STM32 boards USART1 (PA9/PA10).

Co-Authored-By: Claude Sonnet 5.5 <noreply@anthropic.com>
Parts:
- added J_UART1: UART, Connector_PinHeader_2.54mm:PinHeader_1x03_P2.54mm_Vertical, F.Cu at (77.6, 85.3)
- added TP_SCL: SCL, TestPoint:TestPoint_Pad_D1.5mm, F.Cu at (69.1, 87.2)
- added TP_SDA: SDA, TestPoint:TestPoint_Pad_D1.5mm, F.Cu at (66.5, 87.2)
Connections:
- U_MCU pad 19: unconnected-(U_MCU-PA9-Pad19) -> UART_TX
- U_MCU pad 21: unconnected-(U_MCU-PA10-Pad21) -> UART_RX
Routing:
- net SCL_EXT: track 52.1 -> 73.7 mm
- net SDA_EXT: track 55.3 -> 76.4 mm, vias 2 -> 1
- net SYS_CHG: track 43.8 -> 27.4 mm, vias 3 -> 2
- net UART_RX: track 0.00 -> 16.0 mm
- net SW3_G: track 42.2 -> 56.4 mm
- net CHG_CE: track 83.7 -> 97.4 mm, vias 4 -> 2
- net SNS_S4: track 68.3 -> 81.9 mm
- net UART_TX: track 0.00 -> 12.8 mm
- net MON_PWRDN: track 61.7 -> 74.4 mm, vias 3 -> 5
- net SW3_DRV: track 65.0 -> 77.6 mm, vias 4 -> 2
- net MON_ALERT: track 57.9 -> 70.1 mm
- net FB: track 24.5 -> 35.7 mm, vias 2 -> 0
- net SYS: track 94.1 -> 83.5 mm
- net NRST: track 65.0 -> 55.2 mm
- net REGN: track 33.8 -> 43.3 mm, vias 2 -> 4
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Other:
- board text added: "GND TX RX"
- board text added: "SCL"
- board text added: "SDA"

Commit message: hardware: KiCad 10 pipeline fixes, +5V reservoir caps, NS4168 1uF, pack UART header off the holders
KiCad 9 -> 10.0.7 broke the generators even on HEAD:
- gen_sch: libraries moved (hide yes) from effects to the property; read both,
  write it back into effects (KiCad 9 format), so hidden fields stop showing
  on every sheet and stop blocking the schematic router. Add the title block.
- gen_pcb: SetDoNotAllowCopperPour -> SetDoNotAllowZoneFills; copy the symbol's
  Datasheet/Description/Sim fields onto footprints (schematic parity now fails
  DRC); refuse THT pads under bottom-side parts (PTH_UNDER_OK allowlist).
- route.py: Power class routed at +40 um (Freerouting's octagons undercut 0.8 mm
  round ends, KiCad 10 exports no clearance margin), falling back to no margin
  if that leaves a connection unrouted; strip dangling stubs after SES import.
- pack: USB-C shield pin S1 -> SH; pack_tme: VSSOP-10 -> MSOP-10 footprint.

Design changes from the Konnect MCP review and datasheet check:
- carrier: C_5V1 10 uF + C_5V2 100 nF on +5V at J_PWR1 (no local cap before);
  C_AMP2 100 nF -> 1 uF per NS4168 datasheet (100 uF || 1 uF). carrier_tme
  places the new caps clear of its DAC.
- pack/pack_tme: J_UART1 sat under BT4 (bottom-side 18650 holder), caught by
  KiCad 10's pth_inside_courtyard; moved to the right strip, label in pin order.
  The NTC beads stay in the holder window (check ignored, gen_pcb enforces it).
- Docs: ORDERING counts, NS4168/TCA9534/BSS138/1N4148W datasheet check,
  TCA9534 P6/P7 firmware note.

All six boards: ERC 0, DRC 0 (0 unconnected, 0 parity), gerbers ok.

Co-Authored-By: Claude Opus 5.5 <noreply@anthropic.com>
Parts:
- moved J_UART1 18.8 mm to (88.5, 70.0), turned to 180 degrees
Routing:
- net CHG_INT: track 74.3 -> 98.1 mm
- net USB_DM: track 88.9 -> 67.7 mm
- net CHG_CE: track 97.4 -> 79.6 mm, vias 2 -> 3
- net NTC1: track 85.5 -> 103.3 mm
- net +5V: track 41.3 -> 57.6 mm, vias 1 -> 2
- net SW3_G: track 56.4 -> 42.5 mm
- net SDA_INT: track 89.4 -> 76.0 mm, vias 5 -> 6
- net FB: track 35.7 -> 25.2 mm, vias 0 -> 2
- net UART_TX: track 12.8 -> 22.9 mm
- net KEY_OUT: track 34.1 -> 43.6 mm
- net BAT_CHG: track 16.4 -> 25.9 mm, vias 2 -> 3
- net SW4_DRV: track 63.0 -> 53.7 mm
- net REGN: track 43.3 -> 34.2 mm, vias 4 -> 2
- net SW2_G: track 42.4 -> 51.1 mm, vias 0 -> 2
- net SW4_G: track 41.0 -> 49.7 mm, vias 0 -> 2
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