File: hardware/kicad/pack_tme.kicad_pcb (KiCad board)
At the start: 2 copper layers, 96 x 90 mm, 129 parts, among them U1 MCP1640T-I/CHY

Commit message: hardware: UART debug header on all boards, I2C header and rail test pads on carrier, SDA/SCL pads on pack
Header is 1x3 2.54 mm (GND, MCU TX, MCU RX), hand-soldered, kept out of the BOM.
Carrier uses Heltec UART0 (GPIO43/44), STM32 boards USART1 (PA9/PA10).

Co-Authored-By: Claude Sonnet 5.5 <noreply@anthropic.com>
Parts:
- added J_UART1: UART, Connector_PinHeader_2.54mm:PinHeader_1x03_P2.54mm_Vertical, F.Cu at (78.4, 79.0)
- added TP_SCL: SCL, TestPoint:TestPoint_Pad_D1.5mm, F.Cu at (68.8, 87.4)
- added TP_SDA: SDA, TestPoint:TestPoint_Pad_D1.5mm, F.Cu at (66.0, 87.4)
Connections:
- U_MCU pad 19: unconnected-(U_MCU-PA9-Pad19) -> UART_TX
- U_MCU pad 20: unconnected-(U_MCU-PA10-Pad20) -> UART_RX
Routing:
- net SYS: track 84.9 -> 118.7 mm
- net CELL2_SRC: track 14.4 -> 47.0 mm
- net SDA_EXT: track 33.4 -> 64.9 mm
- net SCL_EXT: track 32.7 -> 60.7 mm, vias 2 -> 3
- net SW_CHG: track 41.2 -> 63.1 mm
- net VBUS: track 54.6 -> 71.2 mm
- net SCL_INT: track 141.5 -> 158.1 mm
- net GND: track 639.2 -> 654.8 mm, vias 0 -> 8
- net +3V3: track 249.3 -> 264.3 mm, vias 6 -> 7
- net NTC2: track 55.5 -> 69.9 mm
- net BOOT0: track 95.7 -> 109.1 mm, vias 2 -> 3
- net CHG_CE: track 94.7 -> 107.6 mm
- net SW2_DRV: track 98.6 -> 86.2 mm, vias 2 -> 6
- net SW1_DRV: track 101.6 -> 112.8 mm
- net UART_RX: track 0.00 -> 10.9 mm, vias 0 -> 1
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Other:
- board text added: "GND TX RX"
- board text added: "SCL"
- board text added: "SDA"

Commit message: hardware: KiCad 10 pipeline fixes, +5V reservoir caps, NS4168 1uF, pack UART header off the holders
KiCad 9 -> 10.0.7 broke the generators even on HEAD:
- gen_sch: libraries moved (hide yes) from effects to the property; read both,
  write it back into effects (KiCad 9 format), so hidden fields stop showing
  on every sheet and stop blocking the schematic router. Add the title block.
- gen_pcb: SetDoNotAllowCopperPour -> SetDoNotAllowZoneFills; copy the symbol's
  Datasheet/Description/Sim fields onto footprints (schematic parity now fails
  DRC); refuse THT pads under bottom-side parts (PTH_UNDER_OK allowlist).
- route.py: Power class routed at +40 um (Freerouting's octagons undercut 0.8 mm
  round ends, KiCad 10 exports no clearance margin), falling back to no margin
  if that leaves a connection unrouted; strip dangling stubs after SES import.
- pack: USB-C shield pin S1 -> SH; pack_tme: VSSOP-10 -> MSOP-10 footprint.

Design changes from the Konnect MCP review and datasheet check:
- carrier: C_5V1 10 uF + C_5V2 100 nF on +5V at J_PWR1 (no local cap before);
  C_AMP2 100 nF -> 1 uF per NS4168 datasheet (100 uF || 1 uF). carrier_tme
  places the new caps clear of its DAC.
- pack/pack_tme: J_UART1 sat under BT4 (bottom-side 18650 holder), caught by
  KiCad 10's pth_inside_courtyard; moved to the right strip, label in pin order.
  The NTC beads stay in the holder window (check ignored, gen_pcb enforces it).
- Docs: ORDERING counts, NS4168/TCA9534/BSS138/1N4148W datasheet check,
  TCA9534 P6/P7 firmware note.

All six boards: ERC 0, DRC 0 (0 unconnected, 0 parity), gerbers ok.

Co-Authored-By: Claude Opus 5.5 <noreply@anthropic.com>
Parts:
- U_MON1, U_MON2, U_MON3, U_MON4: footprint Package_SO:VSSOP-10_3x3mm_P0.5mm -> Package_SO:MSOP-10_3x3mm_P0.5mm
- moved J_UART1 30.0 mm to (92.5, 52.5), turned to 180 degrees
Routing:
- net VBAT_SW: track 62.6 -> 101.7 mm, vias 2 -> 0
- net UART_RX: track 10.9 -> 40.5 mm
- net UART_TX: track 9.47 -> 38.8 mm, vias 0 -> 1
- net SYS: track 118.7 -> 89.9 mm, vias 2 -> 4
- net CELL2_SRC: track 47.0 -> 19.9 mm, vias 2 -> 3
- net SW1_DRV: track 112.8 -> 94.5 mm, vias 2 -> 4
- net +3V3: track 264.3 -> 281.8 mm, vias 7 -> 6
- net GND: track 654.8 -> 639.9 mm, vias 8 -> 12
- net SNS_S4: track 27.4 -> 41.3 mm
- net USB_DP: track 79.3 -> 66.1 mm, vias 3 -> 1
- net NRST: track 98.0 -> 111.2 mm, vias 2 -> 4
- net NTC2: track 69.9 -> 57.3 mm, vias 2 -> 1
- net NTC3: track 32.6 -> 45.0 mm, vias 2 -> 1
- net MON_ALERT: track 115.0 -> 127.2 mm
- net SDA_INT: track 159.4 -> 147.2 mm
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