File: hardware/kicad/lipo_tme.kicad_sch (KiCad schematic)
At the start: 63 parts

Commit message: hardware: lipo_tme hierarchical schematic (derived from lipo)
lipo_tme derives its SHEETS/ROOT/OFFBOARD from lipo.py by import and edit,
the way it already derives PARTS/NETS/BLOCKS: lipo's sheets, root and
off-board parts, with the buck sheet titled for the TPS563200 (4.07 V /
5.05 V) and the MCU sheet for the STM32L072. The L072's dedicated BOOT0 test
pad is a root part in the bring-up row, at the same 15.24 mm pitch as lipo's
pads.

make BOARD=lipo_tme all: netlist matches lipo_tme.py, ERC 0, DRC 0
violations / 0 unconnected / 0 schematic parity, gerbers ok. Board unchanged
apart from footprint paths (tools/pcb_diff.py --allow-unnamed against
596060b: 63 footprints, 43 changed path). Konnect
check_schematic_overlaps 0 on all 6 files; run_design_review on root + board
0 errors (8 warnings: 4 MPN and the U_MCU NRST pull-up from the flat
baseline, plus #X_CARRIER I2C pull-ups on the carrier and mcu +3V3 bulk on
the root).
Parts:
- removed C_BTA, C_BTB, C_MCU1, C_MCU3, C_NRST, C_TAP1, C_TAP2, C_TAP3: 100nF, Capacitor_SMD:C_0805_2012Metric_Pad1.18x1.45mm_HandSolder, symbol Device:C
- removed C_LDO1, C_VIN2, C_VIN3, C_VIN4: 10uF, Capacitor_SMD:C_0805_2012Metric_Pad1.18x1.45mm_HandSolder, symbol Device:C
- removed C_MCU2: 4u7, Capacitor_SMD:C_0805_2012Metric_Pad1.18x1.45mm_HandSolder, symbol Device:C
- removed C_OA1, C_OB1: 22uF 25V, Capacitor_SMD:C_1206_3216Metric_Pad1.33x1.80mm_HandSolder, symbol Device:C
- removed C_VDDA: 1uF, Capacitor_SMD:C_0805_2012Metric_Pad1.18x1.45mm_HandSolder, symbol Device:C
- removed D_GZ1: MMSZ5240B, Diode_SMD:D_SOD-123, symbol Device:D_Zener
- removed D_TVS1: SMBJ15A, Diode_SMD:D_SMB, symbol Device:D_Zener
- removed F_IN1: 5A fuse, Fuse:Fuse_1206_3216Metric_Pad1.42x1.75mm_HandSolder, symbol Device:Fuse
- removed L_A, L_B: 3u3, Inductor_SMD:L_Bourns_SRN6045TA, symbol Device:L
- removed Q_KILL: BSS138, Package_TO_SOT_SMD:SOT-23, symbol Transistor_FET:BSS138
- removed Q_REV1: AO3401A, Package_TO_SOT_SMD:SOT-23, symbol Transistor_FET:AO3401A
- removed R_BOOT, R_FBB2: 10k, Resistor_SMD:R_0805_2012Metric_Pad1.20x1.40mm_HandSolder, symbol Device:R
- removed R_EN2: 47k, Resistor_SMD:R_0805_2012Metric_Pad1.20x1.40mm_HandSolder, symbol Device:R
- removed R_FBA1: 22k, Resistor_SMD:R_0805_2012Metric_Pad1.20x1.40mm_HandSolder, symbol Device:R
- removed R_FBA2: 5k1, Resistor_SMD:R_0805_2012Metric_Pad1.20x1.40mm_HandSolder, symbol Device:R
- removed R_FBB1: 56k, Resistor_SMD:R_0805_2012Metric_Pad1.20x1.40mm_HandSolder, symbol Device:R
- removed R_GK, R_REV1: 100k, Resistor_SMD:R_0805_2012Metric_Pad1.20x1.40mm_HandSolder, symbol Device:R
- removed R_KILL: 1k, Resistor_SMD:R_0805_2012Metric_Pad1.20x1.40mm_HandSolder, symbol Device:R
- removed R_TB1, R_TT2, R_TT3, R_TT3B: 1M, Resistor_SMD:R_0805_2012Metric_Pad1.20x1.40mm_HandSolder, symbol Device:R
- removed R_TB2, R_TB3, R_TT1: 470k, Resistor_SMD:R_0805_2012Metric_Pad1.20x1.40mm_HandSolder, symbol Device:R
- removed U_BA, U_BB: TPS563200DDCR, Package_TO_SOT_SMD:TSOT-23-6, symbol Regulator_Switching:TPS563200
- removed U_LDO: AP7381-33SA-7, Package_TO_SOT_SMD:SOT-23, symbol Regulator_Linear:AP7381-33SA-7
- removed U_MCU: STM32L072KZT6, Package_QFP:LQFP-32_7x7mm_P0.8mm, symbol MCU_ST_STM32L0:STM32L072KZTx
- added #X_BAL: 2S/3S balance plug, symbol local:Conn_W_04
- added #X_CARRIER: Carrier board (J_PWR1), symbol local:Pack_Link_6
- added #X_KEY: Airsoft key switch, symbol local:Conn_W_02
- added #X_LIPO: 2S/3S LiPo pack, symbol local:Conn_W_02
- J_BAL1: symbol Connector_Generic:Conn_01x04 -> local:Conn_W_04
- J_IN1, J_KEY1: symbol Connector_Generic:Conn_01x02 -> local:Conn_W_02
- J_PWR1: symbol Connector_Generic:Conn_01x06 -> local:Conn_W_06
Connections:
- net +5V: now also #X_CARRIER.4 (5V)
- net BAL1: now also #X_BAL.2
- net BAL2: now also #X_BAL.3
- net BAL3: now also #X_BAL.4
- net BUCK_EN: now also #X_KEY.2
- net GND: now also #X_BAL.1, #X_CARRIER.1 (GND), #X_CARRIER.2 (GND), #X_LIPO.2
- net KEY_IN: now also #X_KEY.1
- net LIPO_RAW: now also #X_LIPO.1
- net SCL_EXT: now also #X_CARRIER.6 (SCL)
- net SDA_EXT: now also #X_CARRIER.5 (SDA)
- net VBAT_SW: now also #X_CARRIER.3 (VBAT)
- no-connect marks 15 -> 0
Other:
- added sheet Always-on 3V3 and STM32L072 (lipo_tme-mcu.kicad_sch)
- added sheet Balance lead dividers (lipo_tme-bal.kicad_sch)
- added sheet Buck A 4.07 V (VBAT_SW), buck B 5.05 V (+5V) (lipo_tme-bucks.kicad_sch)
- added sheet Key enable and MCU kill (lipo_tme-enable.kicad_sch)
- added sheet LiPo input: fuse, reverse FET, TVS (lipo_tme-input.kicad_sch)
- note added: "2S/3S LiPo pack"
- note added: "XH-2"
- note added: "XH-4, 2S plug on pins 1-3"
- note added: "XH-6 to the carrier"
- note added: "XT60 pigtail into the J_IN1 pads"
- note removed: "Always-on 3V3, STM32L072, SWD pads"
- note removed: "Balance lead dividers"
- note removed: "Buck A 4.10 V (VBAT_SW), buck B 5.07 V (+5V)"
- note removed: "Key enable, MCU kill, J_PWR1"
- note removed: "LiPo input: fuse, reverse FET, TVS"
- note removed: "Mounting holes and power flags"
- title: AirsoftCounter v2 LiPo (hand-build) -> AirsoftCounter v2 LiPo (hand-build): system
- moved on the sheet: C_LDO2, C_OA2, C_OB2, C_VIN1, H1, H2, H3, H4, J_UART1, R_EN1, TP_3V3, TP_BOOT0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
