File: hardware/kicad/pack_xiao-cell2.kicad_sch (KiCad schematic)
At the start: 17 parts

Commit message: hardware: TME cost cuts (3 fewer resistor tapes, leaner spares); route.py survives KiCad 10's SWIG break
carrier_tme: R_OL/R_OR 470R -> 1k (DAC RC corner 72 kHz), R_LLB1/R_LLR1 0R -> 10R (button LEDs
have their own resistors). pack_xiao: R_GS1..4 1M -> 240k (17 uA per closed switch). Drops the
0805 0R, 470R and 1M tapes. tme_all: 1206 caps and the 0603 NTC get +10 % spares, no minimum 5.
About -44 PLN on the 5+5 order (order_35742850 prices).

route.py: stub_free moves from --finish to --import. Its connectivity rebuilds broke the SWIG type
table for the rest of the process, so finish() got bare SwigPyObjects for zones (carrier_tme
segfaulted in apport's excepthook on the AttributeError). Placement unchanged on both boards.

Co-Authored-By: Claude Opus 5.5 <noreply@anthropic.com>
Parts:
- R_GS2: value 1M -> 240k
Changed lines of the file:
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@@
 			)
 		)
-		(property "Value" "1M"
+		(property "Value" "240k"
 			(at 43.18 115.57 90)
 			(show_name no)
