File: hardware/kicad/pack_xiao-mcu.kicad_sch (KiCad schematic)
At the start: 7 parts

Commit message: hardware: pack_xiao iron-only (plated holes under XIAO pads 16/20) and fits the enclosure (notch + cutout for the carrier posts)
Footprint XIAO_ESP32S3_SMD_THB (derived by tools/import_xiao.py) makes the two used bottom pads
plated holes, soldered from the board's back. gen_pcb learns NOTCH_BL and CUTOUTS (with a
no-copper fence, the router ignores edge clearance on inner circles); pack_xiao check_posts()
holds them to mech/params. make mech also gates --boards pack_xiao,carrier.

Co-Authored-By: Claude Opus 5.5 <noreply@anthropic.com>
Parts:
- U_MCU: footprint local:XIAO_ESP32S3_SMD -> local:XIAO_ESP32S3_SMD_THB
Changed lines of the file:
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@@
 			)
 		)
-		(property "Footprint" "local:XIAO_ESP32S3_SMD"
+		(property "Footprint" "local:XIAO_ESP32S3_SMD_THB"
 			(at 75.438 94.742 0)
 			(hide yes)

Commit message: hardware: cheaper TME equivalents; THB footprint in its own library; per-board KIID seed
TME swaps (user-picked, checked against each part's job): BSS138LT1G -> BSS138A-TP (all boards),
ERJ8BWFR010V -> Wayon MBR1206B5FR010S shunt, NTCS0603E3103FLT -> Murata NCU18XH103J6SRB (TH_CHG,
B3380 5 %: ~+-1.5 C on the charger limits), pack_xiao boost caps 22uF 25V -> CL31A226MOCLNNC 16 V
(5 V max; the LiPo keeps its 25 V parts).

Adding XIAO_ESP32S3_SMD_THB to local.pretty had renumbered every board using that library (KiCad
parses the whole library on first load, drawing on the seeded KIID sequence): pack_tme's footprint
order changed and Freerouting left a connection unrouted. The footprint moves to kicad/xiao.pretty;
pack_tme routes as before. gen_pcb takes KIID_SEED per board (default 1); pack_xiao uses 2.

Co-Authored-By: Claude Opus 5.5 <noreply@anthropic.com>
Parts:
- U_MCU: footprint local:XIAO_ESP32S3_SMD_THB -> xiao:XIAO_ESP32S3_SMD_THB
Changed lines of the file:
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@@
 			)
 		)
-		(property "Footprint" "local:XIAO_ESP32S3_SMD_THB"
+		(property "Footprint" "xiao:XIAO_ESP32S3_SMD_THB"
 			(at 75.438 94.742 0)
 			(hide yes)
