File: hardware/kicad/pack_xiao.kicad_sch (KiCad schematic)
At the start: 19 parts, among them U1 MCP1640T-I/CHY

Commit message: hardware: cheaper TME equivalents; THB footprint in its own library; per-board KIID seed
TME swaps (user-picked, checked against each part's job): BSS138LT1G -> BSS138A-TP (all boards),
ERJ8BWFR010V -> Wayon MBR1206B5FR010S shunt, NTCS0603E3103FLT -> Murata NCU18XH103J6SRB (TH_CHG,
B3380 5 %: ~+-1.5 C on the charger limits), pack_xiao boost caps 22uF 25V -> CL31A226MOCLNNC 16 V
(5 V max; the LiPo keeps its 25 V parts).

Adding XIAO_ESP32S3_SMD_THB to local.pretty had renumbered every board using that library (KiCad
parses the whole library on first load, drawing on the seeded KIID sequence): pack_tme's footprint
order changed and Freerouting left a connection unrouted. The footprint moves to kicad/xiao.pretty;
pack_tme routes as before. gen_pcb takes KIID_SEED per board (default 1); pack_xiao uses 2.

Co-Authored-By: Claude Opus 5.5 <noreply@anthropic.com>
Parts:
- C_IN1, C_OUT1, C_OUT2: value 22uF 25V -> 22uF 16V
Changed lines of the file:
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@@
 			)
 		)
-		(property "Value" "22uF 25V"
+		(property "Value" "22uF 16V"
 			(at 206.375 38.1 0)
 			(show_name no)
@@
 			)
 		)
-		(property "Value" "22uF 25V"
+		(property "Value" "22uF 16V"
 			(at 127.635 53.34 0)
 			(show_name no)
@@
 			)
 		)
-		(property "Value" "22uF 25V"
+		(property "Value" "22uF 16V"
 			(at 216.535 48.26 0)
 			(show_name no)
