File: hardware/kicad/carrier.kicad_sch (KiCad schematic)
At the start: 40 parts, among them J2 Heltec_J2, J3 Heltec_J3

Commit message: hardware: 3.5" ILI9488 SPI TFT replaces the Newhaven LCD
Carrier and carrier_tme: J_LCD1 XH-8 (VCC GND CS RST DC MOSI SCK LED,
the module header order; CS tied low). SPI3 on GPIO43/44, PWM backlight
on GPIO6 (R_BLPD1), DC/RST on TCA9534 P6/P7, buttons polled. The P4/P5
native-pin option was dropped: the Heltec GNSS receptacle opens toward
those pins. Removed the I2C level shifter, R_INT1/EXP_INT and J_UART1;
J_NFC1 moved to the bottom edge. Both boards: 0 unrouted, ERC/DRC/parity 0.

Lid rebuilt from the LCDWiki MSP3520 drawing: 98 x 56.34, M3 bosses on
92 x 49.5 (r3.0, 4.5 high), 80 x 51 viewing window, 11.5 mm depth.
make mech green. Power model: backlight duty is now the mean PWM level.

Co-Authored-By: Claude Opus 5.5 <noreply@anthropic.com>
Parts:
- removed J_UART1: UART, Connector_PinHeader_2.54mm:PinHeader_1x03_P2.54mm_Vertical, symbol Connector_Generic:Conn_01x03
- removed Q_SCL1, Q_SDA1: BSS138, Package_TO_SOT_SMD:SOT-23, symbol Transistor_FET:BSS138
- removed R_SCL5, R_SDA5: 4k7, Resistor_SMD:R_0805_2012Metric_Pad1.20x1.40mm_HandSolder, symbol Device:R
- added R_BLPD1: 10k, Resistor_SMD:R_0805_2012Metric_Pad1.20x1.40mm_HandSolder, symbol Device:R
- #X_LCD: value LCD 1602 + PCF8574 -> 3.5" ILI9488 SPI TFT; symbol local:Module_I2C_4 -> local:Conn_W_08
- J_LCD1: footprint Connector_JST:JST_XH_B4B-XH-A_1x04_P2.50mm_Vertical -> Connector_JST:JST_XH_B8B-XH-A_1x08_P2.50mm_Vertical; symbol local:Conn_W_04 -> local:Conn_W_08
Connections:
- net SDA_5V is gone; now on net GND: #X_LCD.3, J_LCD1.3
- net +5V: now also #X_LCD.1, J_LCD1.1; no longer #X_LCD.2 (VCC), J_LCD1.2
- net GND: now also #X_LCD.2, J_LCD1.2, R_BLPD1.2; no longer #X_LCD.1 (GND), J_LCD1.1
- net EXP_INT renamed LCD_BL
- net LCD_BL: now also #X_LCD.8, J_LCD1.8, R_BLPD1.1
- net SCL_5V renamed LCD_RST
- net UART_RX renamed LCD_MOSI
- net LCD_MOSI: now also #X_LCD.6, J_LCD1.6
- net UART_TX renamed LCD_SCK
- net LCD_SCK: now also #X_LCD.7, J_LCD1.7
- new net LCD_DC: #X_LCD.5, J_LCD1.5
Other:
- sheet GPIO expander (0x20), button inputs ports: added LCD_DC, LCD_RST; removed EXP_INT
- note added: "XH-8, straight"
