File: hardware/kicad/carrier_tme-drivers.kicad_sch (KiCad schematic)
At the start: 12 parts

Commit message: hardware: carrier_tme schematic: cables, root board-edge parts, review clean
Review (Konnect, audits each sheet on its own): 20 errors -> 0.
- Off-board parts are virtual #X_* symbols (out of the netlist and BOMs).
- Board-edge parts are drawn on the root beside their connectors: the
  power-entry caps, the debug headers and test pads, D_FLY1 (across the
  buzzer) and the I2C level shifter with the bus pull-ups. Every rail on the
  root has its bulk cap there; the i2c, power and debug sheets are gone
  (function sheets: expander, drivers, audio).
- J2 pin 2 is "CHG IN" (a 5V name read as an undecoupled supply pin).

Cables: root connectors and off-board modules use 5.08 mm-pitch symbols
(local:Conn_W_02/04/06, recreated module symbols; footprints unchanged).
Every off-board pin is wired to its connector pin; a rail's power port hangs
off its cable (gen_sch cable + tee_port, drawn after the signals). 2.54 mm
headers keep ports along their stubs (ROOT port_modes).

Leftover gaps: gen_sch fits each function block to its content.

make BOARD=carrier_tme all: netlist matches, ERC 0, DRC 0/0/0 parity,
gerbers ok; board changed only in footprint paths and J2's unconnected net
name. Flat boards regenerate byte-identical. Remaining review warnings: MPN,
U2 pull-ups and expander bulk (both on the root sheet).

Co-Authored-By: Claude Opus 5.5 <noreply@anthropic.com>
Parts:
- removed D_FLY1: 1N4148W, Diode_SMD:D_SOD-123, symbol Diode:1N4148W
Other:
- moved on the sheet: Q_BZ1, Q_LB1, Q_LR1, R_GBZ1, R_GLB1, R_GLR1, R_LLB1, R_LLR1, R_PDBZ1, R_PDLB1, R_PDLR1

Commit message: hardware: TME cost cuts (3 fewer resistor tapes, leaner spares); route.py survives KiCad 10's SWIG break
carrier_tme: R_OL/R_OR 470R -> 1k (DAC RC corner 72 kHz), R_LLB1/R_LLR1 0R -> 10R (button LEDs
have their own resistors). pack_xiao: R_GS1..4 1M -> 240k (17 uA per closed switch). Drops the
0805 0R, 470R and 1M tapes. tme_all: 1206 caps and the 0603 NTC get +10 % spares, no minimum 5.
About -44 PLN on the 5+5 order (order_35742850 prices).

route.py: stub_free moves from --finish to --import. Its connectivity rebuilds broke the SWIG type
table for the rest of the process, so finish() got bare SwigPyObjects for zones (carrier_tme
segfaulted in apport's excepthook on the AttributeError). Placement unchanged on both boards.

Co-Authored-By: Claude Opus 5.5 <noreply@anthropic.com>
Parts:
- R_LLB1, R_LLR1: value 0R -> 10R
Changed lines of the file:
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@@
 			)
 		)
-		(property "Value" "0R"
+		(property "Value" "10R"
 			(at 69.85 36.83 90)
 			(show_name no)
@@
 			)
 		)
-		(property "Value" "0R"
+		(property "Value" "10R"
 			(at 128.27 36.83 90)
 			(show_name no)
