File: hardware/kicad/carrier_tme.kicad_sch (KiCad schematic)
At the start: 73 parts, among them J2 Heltec_J2, J3 Heltec_J3, U2 TCA9534PWR

Commit message: hardware: carrier_tme hierarchical schematic
carrier_tme is now a 7-page hierarchy: a system sheet (Heltec V4 with named
pins, every connector, the off-board parts with cable notes, function sheet
boxes wired to the GPIOs) plus power, I2C shifter, expander + buttons,
drivers, DAC + amp and debug sheets.

make BOARD=carrier_tme all: netlist matches carrier_tme.py, ERC 0, DRC 0 /
0 unconnected / 0 schematic parity, gerbers ok. The board differs from the
previous one only in footprint paths (59 sheet parts) and J2/J3's
unconnected-pin net names (named pins); placement, pad nets, routing, BOM and
TME lists unchanged. The flat boards regenerate with no changes.

Co-Authored-By: Claude Opus 5.5 <noreply@anthropic.com>
Parts:
- removed C_5V1, C_DBULK: 10uF, Capacitor_SMD:C_0805_2012Metric_Pad1.18x1.45mm_HandSolder, symbol Device:C
- removed C_5V2, C_BB1, C_BR1, C_DAVDD, C_DCPV, C_DLDO, C_DVDD, C_EXP1: 100nF, Capacitor_SMD:C_0805_2012Metric_Pad1.18x1.45mm_HandSolder, symbol Device:C
- removed C_AMP1, C_NFC1: 100uF 6.3V, Capacitor_SMD:C_1206_3216Metric_Pad1.33x1.80mm_HandSolder, symbol Device:C
- removed C_AMP2, C_INN, C_INP: 1uF, Capacitor_SMD:C_0805_2012Metric_Pad1.18x1.45mm_HandSolder, symbol Device:C
- removed C_BULK1, C_BULK2: 47uF 10V, Capacitor_SMD:C_1206_3216Metric_Pad1.33x1.80mm_HandSolder, symbol Device:C
- removed C_DCP, C_DNEG: 2.2uF, Capacitor_SMD:C_0805_2012Metric_Pad1.18x1.45mm_HandSolder, symbol Device:C
- removed C_OL, C_OR: 2.2nF, Capacitor_SMD:C_0805_2012Metric_Pad1.18x1.45mm_HandSolder, symbol Device:C
- removed D_FLY1: 1N4148W, Diode_SMD:D_SOD-123, symbol Diode:1N4148W
- removed J_I2C1: I2C, Connector_PinHeader_2.54mm:PinHeader_1x04_P2.54mm_Vertical, symbol Connector_Generic:Conn_01x04
- removed J_UART1: UART, Connector_PinHeader_2.54mm:PinHeader_1x03_P2.54mm_Vertical, symbol Connector_Generic:Conn_01x03
- removed Q_BZ1, Q_LB1, Q_LR1, Q_SCL1, Q_SDA1: BSS138, Package_TO_SOT_SMD:SOT-23, symbol Transistor_FET:BSS138
- removed R_GBZ1, R_GLB1, R_GLR1, R_SB1, R_SD1, R_SR1: 1k, Resistor_SMD:R_0805_2012Metric_Pad1.20x1.40mm_HandSolder, symbol Device:R
- removed R_INN, R_INP: 240k, Resistor_SMD:R_0805_2012Metric_Pad1.20x1.40mm_HandSolder, symbol Device:R
- removed R_INT1, R_PDBZ1, R_PDLB1, R_PDLR1, R_PUB1, R_PUR1, R_SDPD1: 10k, Resistor_SMD:R_0805_2012Metric_Pad1.20x1.40mm_HandSolder, symbol Device:R
- removed R_LLB1, R_LLR1: 0R, Resistor_SMD:R_0805_2012Metric_Pad1.20x1.40mm_HandSolder, symbol Device:R
- removed R_OL, R_OR: 470R, Resistor_SMD:R_0805_2012Metric_Pad1.20x1.40mm_HandSolder, symbol Device:R
- removed R_SCL3, R_SCL5, R_SDA3, R_SDA5: 4k7, Resistor_SMD:R_0805_2012Metric_Pad1.20x1.40mm_HandSolder, symbol Device:R
- removed TP_3V3: 3V3, TestPoint:TestPoint_Pad_D1.5mm, symbol Connector:TestPoint
- removed TP_5V: 5V, TestPoint:TestPoint_Pad_D1.5mm, symbol Connector:TestPoint
- removed TP_GND: GND, TestPoint:TestPoint_Pad_D1.5mm, symbol Connector:TestPoint
- removed TP_VSW: VBAT_SW, TestPoint:TestPoint_Pad_D1.5mm, symbol Connector:TestPoint
- removed U2: TCA9534PWR, Package_SO:TSSOP-16_4.4x5mm_P0.65mm, symbol Interface_Expansion:TCA9534
- removed U_AMP: PAM8302AADCR, Package_SO:SOIC-8_3.9x4.9mm_P1.27mm, symbol Amplifier_Audio:PAM8302AAD
- removed U_DAC: PCM5100APWR, Package_SO:TSSOP-20_4.4x6.5mm_P0.65mm, symbol Audio:PCM5100A
- added X_BTN_B: ONPOW LAS1-AGQ-11E/B/6V, symbol local:Button_LED_4
- added X_BTN_R: ONPOW LAS1-AGQ-11E/R/6V, symbol local:Button_LED_4
- added X_BUZ: BZ-38 buzzer, symbol Device:Buzzer
- added X_HBAT: Heltec V4 battery, symbol Connector_Generic:Conn_01x02
- added X_LCD: LCD 1602 + PCF8574, symbol local:Module_I2C_4
- added X_NFC: PN532 (I2C), symbol local:Module_I2C_4
- added X_PACK: Pack board (P5), symbol local:Pack_Link_6
- added X_SPK: VISATON K 50, 8 ohm, symbol Device:Speaker
- J2: symbol Connector_Generic:Conn_01x18 -> local:Heltec_V4_J2
- J3: symbol Connector_Generic:Conn_01x18 -> local:Heltec_V4_J3
Connections:
- net +3V3: now also X_NFC.2 (VCC)
- net +5V: now also X_BTN_B.3 (LED+), X_BTN_R.3 (LED+), X_BUZ.1 (+), X_LCD.2 (VCC), X_PACK.4 (5V)
- net BTN_B_LEDK: now also X_BTN_B.4 (LED-)
- net BTN_B_SW: now also X_BTN_B.1 (SW)
- net BTN_R_LEDK: now also X_BTN_R.4 (LED-)
- net BTN_R_SW: now also X_BTN_R.1 (SW)
- net BUZ_K: now also X_BUZ.2 (-)
- net GND: now also X_BTN_B.2 (COM), X_BTN_R.2 (COM), X_HBAT.2 (Pin_2), X_LCD.1 (GND), X_NFC.1 (GND), X_PACK.1 (GND), X_PACK.2 (GND)
- net SCL_3V3: now also X_NFC.4 (SCL), X_PACK.6 (SCL)
- net SCL_5V: now also X_LCD.4 (SCL)
- net SDA_3V3: now also X_NFC.3 (SDA), X_PACK.5 (SDA)
- net SDA_5V: now also X_LCD.3 (SDA)
- net SPK_N: now also X_SPK.1
- net SPK_P: now also X_SPK.2
- net VBAT_SW: now also X_HBAT.1 (Pin_1), X_PACK.3 (VBAT)
- no-connect marks 27 -> 24
Other:
- added sheet Debug: UART, I2C, test pads (carrier_tme-debug.kicad_sch)
- added sheet GPIO expander (0x20), button inputs (carrier_tme-expander.kicad_sch)
- added sheet I2C level shifter, NFC bulk (carrier_tme-i2c.kicad_sch)
- added sheet I2S DAC and speaker amp (carrier_tme-audio.kicad_sch)
- added sheet Low-side drivers: button LEDs, buzzer (carrier_tme-drivers.kicad_sch)
- added sheet Power: pack rail bulk, +5V reservoir (carrier_tme-power.kicad_sch)
- note added: "Heltec WiFi LoRa 32 V4 (plugs into J2/J3)"
- note added: "XH-2"
- note added: "XH-2 to the module's SH1.25"
- note added: "XH-2, BTL: neither side is GND"
- note added: "XH-4"
- note added: "XH-6"
- note removed: "Debug: UART, I2C, test pads"
- note removed: "GPIO expander (0x20), button inputs"
- note removed: "Heltec V4 headers"
- note removed: "I2C level shifter, LCD (5 V), NFC (3.3 V)"
- note removed: "I2S DAC and speaker amp"
- note removed: "Low-side drivers: button LEDs, buzzer"
- note removed: "Mounting holes"
- note removed: "Power in (from pack board)"
- title: AirsoftCounter v2 carrier (hand-build) -> AirsoftCounter v2 carrier (hand-build): system
- moved on the sheet: H1, H2, H3, H4, J2, J3, J_BTN_B1, J_BTN_R1, J_BUZ1, J_HBAT1, J_LCD1, J_NFC1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

Commit message: hardware: carrier_tme schematic: cables, root board-edge parts, review clean
Review (Konnect, audits each sheet on its own): 20 errors -> 0.
- Off-board parts are virtual #X_* symbols (out of the netlist and BOMs).
- Board-edge parts are drawn on the root beside their connectors: the
  power-entry caps, the debug headers and test pads, D_FLY1 (across the
  buzzer) and the I2C level shifter with the bus pull-ups. Every rail on the
  root has its bulk cap there; the i2c, power and debug sheets are gone
  (function sheets: expander, drivers, audio).
- J2 pin 2 is "CHG IN" (a 5V name read as an undecoupled supply pin).

Cables: root connectors and off-board modules use 5.08 mm-pitch symbols
(local:Conn_W_02/04/06, recreated module symbols; footprints unchanged).
Every off-board pin is wired to its connector pin; a rail's power port hangs
off its cable (gen_sch cable + tee_port, drawn after the signals). 2.54 mm
headers keep ports along their stubs (ROOT port_modes).

Leftover gaps: gen_sch fits each function block to its content.

make BOARD=carrier_tme all: netlist matches, ERC 0, DRC 0/0/0 parity,
gerbers ok; board changed only in footprint paths and J2's unconnected net
name. Flat boards regenerate byte-identical. Remaining review warnings: MPN,
U2 pull-ups and expander bulk (both on the root sheet).

Co-Authored-By: Claude Opus 5.5 <noreply@anthropic.com>
Parts:
- removed X_BTN_B: ONPOW LAS1-AGQ-11E/B/6V, symbol local:Button_LED_4
- removed X_BTN_R: ONPOW LAS1-AGQ-11E/R/6V, symbol local:Button_LED_4
- removed X_BUZ: BZ-38 buzzer, symbol Device:Buzzer
- removed X_HBAT: Heltec V4 battery, symbol Connector_Generic:Conn_01x02
- removed X_LCD: LCD 1602 + PCF8574, symbol local:Module_I2C_4
- removed X_NFC: PN532 (I2C), symbol local:Module_I2C_4
- removed X_PACK: Pack board (P5), symbol local:Pack_Link_6
- removed X_SPK: VISATON K 50, 8 ohm, symbol Device:Speaker
- added #X_BTN_B: ONPOW LAS1-AGQ-11E/B/6V, symbol local:Button_LED_4
- added #X_BTN_R: ONPOW LAS1-AGQ-11E/R/6V, symbol local:Button_LED_4
- added #X_BUZ: BZ-38 buzzer, symbol Device:Buzzer
- added #X_HBAT: Heltec V4 battery, symbol local:Conn_W_02
- added #X_LCD: LCD 1602 + PCF8574, symbol local:Module_I2C_4
- added #X_NFC: PN532 (I2C), symbol local:Module_I2C_4
- added #X_PACK: Pack board (P5), symbol local:Pack_Link_6
- added #X_SPK: VISATON K 50, 8 ohm, symbol Device:Speaker
- added C_5V1: 10uF, Capacitor_SMD:C_0805_2012Metric_Pad1.18x1.45mm_HandSolder, symbol Device:C
- added C_5V2: 100nF, Capacitor_SMD:C_0805_2012Metric_Pad1.18x1.45mm_HandSolder, symbol Device:C
- added C_BULK1, C_BULK2: 47uF 10V, Capacitor_SMD:C_1206_3216Metric_Pad1.33x1.80mm_HandSolder, symbol Device:C
- added C_NFC1: 100uF 6.3V, Capacitor_SMD:C_1206_3216Metric_Pad1.33x1.80mm_HandSolder, symbol Device:C
- added D_FLY1: 1N4148W, Diode_SMD:D_SOD-123, symbol Diode:1N4148W
- added J_I2C1: I2C, Connector_PinHeader_2.54mm:PinHeader_1x04_P2.54mm_Vertical, symbol Connector_Generic:Conn_01x04
- added J_UART1: UART, Connector_PinHeader_2.54mm:PinHeader_1x03_P2.54mm_Vertical, symbol Connector_Generic:Conn_01x03
- added Q_SCL1, Q_SDA1: BSS138, Package_TO_SOT_SMD:SOT-23, symbol Transistor_FET:BSS138
- added R_SCL3, R_SCL5, R_SDA3, R_SDA5: 4k7, Resistor_SMD:R_0805_2012Metric_Pad1.20x1.40mm_HandSolder, symbol Device:R
- added TP_3V3: 3V3, TestPoint:TestPoint_Pad_D1.5mm, symbol Connector:TestPoint
- added TP_5V: 5V, TestPoint:TestPoint_Pad_D1.5mm, symbol Connector:TestPoint
- added TP_GND: GND, TestPoint:TestPoint_Pad_D1.5mm, symbol Connector:TestPoint
- added TP_VSW: VBAT_SW, TestPoint:TestPoint_Pad_D1.5mm, symbol Connector:TestPoint
- J_BTN_B1, J_BTN_R1, J_LCD1, J_NFC1: symbol Connector_Generic:Conn_01x04 -> local:Conn_W_04
- J_BUZ1, J_HBAT1, J_SPK1: symbol Connector_Generic:Conn_01x02 -> local:Conn_W_02
- J_PWR1: symbol Connector_Generic:Conn_01x06 -> local:Conn_W_06
Connections:
- net +3V3: now also #X_NFC.2 (VCC), C_NFC1.1, J_I2C1.2 (Pin_2), Q_SCL1.1 (G), Q_SDA1.1 (G), R_SCL3.1, R_SDA3.1, TP_3V3.1
- net +5V: now also #X_BTN_B.3 (LED+), #X_BTN_R.3 (LED+), #X_BUZ.1 (+), #X_LCD.2 (VCC), #X_PACK.4 (5V), C_5V1.1, C_5V2.1, D_FLY1.1 (K), R_SCL5.1, R_SDA5.1, TP_5V.1
- net BTN_B_LEDK: now also #X_BTN_B.4 (LED-)
- net BTN_B_SW: now also #X_BTN_B.1 (SW)
- net BTN_R_LEDK: now also #X_BTN_R.4 (LED-)
- net BTN_R_SW: now also #X_BTN_R.1 (SW)
- net BUZ_K: now also #X_BUZ.2 (-), D_FLY1.2 (A)
- net GND: now also #X_BTN_B.2 (COM), #X_BTN_R.2 (COM), #X_HBAT.2, #X_LCD.1 (GND), #X_NFC.1 (GND), #X_PACK.1 (GND), #X_PACK.2 (GND), C_5V1.2, C_5V2.2, C_BULK1.2, C_BULK2.2, C_NFC1.2, J_I2C1.1 (Pin_1), J_UART1.1 (Pin_1), TP_GND.1
- net SCL_3V3: now also #X_NFC.4 (SCL), #X_PACK.6 (SCL), J_I2C1.4 (Pin_4), Q_SCL1.2 (S), R_SCL3.2
- net SCL_5V: now also #X_LCD.4 (SCL), Q_SCL1.3 (D), R_SCL5.2
- net SDA_3V3: now also #X_NFC.3 (SDA), #X_PACK.5 (SDA), J_I2C1.3 (Pin_3), Q_SDA1.2 (S), R_SDA3.2
- net SDA_5V: now also #X_LCD.3 (SDA), Q_SDA1.3 (D), R_SDA5.2
- net SPK_N: now also #X_SPK.1
- net SPK_P: now also #X_SPK.2
- net UART_RX: now also J_UART1.3 (Pin_3)
- net UART_TX: now also J_UART1.2 (Pin_2)
- net VBAT_SW: now also #X_HBAT.1, #X_PACK.3 (VBAT), C_BULK1.1, C_BULK2.1, TP_VSW.1
Other:
- removed sheet Debug: UART, I2C, test pads
- removed sheet I2C level shifter, NFC bulk
- removed sheet Power: pack rail bulk, +5V reservoir

Commit message: hardware: 3.5" ILI9488 SPI TFT replaces the Newhaven LCD
Carrier and carrier_tme: J_LCD1 XH-8 (VCC GND CS RST DC MOSI SCK LED,
the module header order; CS tied low). SPI3 on GPIO43/44, PWM backlight
on GPIO6 (R_BLPD1), DC/RST on TCA9534 P6/P7, buttons polled. The P4/P5
native-pin option was dropped: the Heltec GNSS receptacle opens toward
those pins. Removed the I2C level shifter, R_INT1/EXP_INT and J_UART1;
J_NFC1 moved to the bottom edge. Both boards: 0 unrouted, ERC/DRC/parity 0.

Lid rebuilt from the LCDWiki MSP3520 drawing: 98 x 56.34, M3 bosses on
92 x 49.5 (r3.0, 4.5 high), 80 x 51 viewing window, 11.5 mm depth.
make mech green. Power model: backlight duty is now the mean PWM level.

Co-Authored-By: Claude Opus 5.5 <noreply@anthropic.com>
Parts:
- removed J_UART1: UART, Connector_PinHeader_2.54mm:PinHeader_1x03_P2.54mm_Vertical, symbol Connector_Generic:Conn_01x03
- removed Q_SCL1, Q_SDA1: BSS138, Package_TO_SOT_SMD:SOT-23, symbol Transistor_FET:BSS138
- removed R_SCL5, R_SDA5: 4k7, Resistor_SMD:R_0805_2012Metric_Pad1.20x1.40mm_HandSolder, symbol Device:R
- added R_BLPD1: 10k, Resistor_SMD:R_0805_2012Metric_Pad1.20x1.40mm_HandSolder, symbol Device:R
- #X_LCD: value LCD 1602 + PCF8574 -> 3.5" ILI9488 SPI TFT; symbol local:Module_I2C_4 -> local:Conn_W_08
- J_LCD1: footprint Connector_JST:JST_XH_B4B-XH-A_1x04_P2.50mm_Vertical -> Connector_JST:JST_XH_B8B-XH-A_1x08_P2.50mm_Vertical; symbol local:Conn_W_04 -> local:Conn_W_08
Connections:
- net SDA_5V is gone; now on net GND: #X_LCD.3, J_LCD1.3
- net +5V: now also #X_LCD.1, J_LCD1.1; no longer #X_LCD.2 (VCC), J_LCD1.2
- net GND: now also #X_LCD.2, J_LCD1.2, R_BLPD1.2; no longer #X_LCD.1 (GND), J_LCD1.1
- net EXP_INT renamed LCD_BL
- net LCD_BL: now also #X_LCD.8, J_LCD1.8, R_BLPD1.1
- net SCL_5V renamed LCD_RST
- net UART_RX renamed LCD_MOSI
- net LCD_MOSI: now also #X_LCD.6, J_LCD1.6
- net UART_TX renamed LCD_SCK
- net LCD_SCK: now also #X_LCD.7, J_LCD1.7
- new net LCD_DC: #X_LCD.5, J_LCD1.5
Other:
- sheet GPIO expander (0x20), button inputs ports: added LCD_DC, LCD_RST; removed EXP_INT
- note added: "XH-8, straight"
