File: hardware/kicad/pack_xiao_jlc-cell1.kicad_sch (KiCad schematic)
At the start: 17 parts

Commit message: hardware(pack_xiao_jlc): hand-solder big-pad Extended parts, 11 -> 4 fee types
No Basic/Preferred fuse, PTC, power inductor or 10 mOhm shunt exists at JLC
(live check 2026-10-28), so the big-pad Extended types leave the JLC BOM:
XH-6/XH-2 connectors, F1-F4, F_SYS1, R_SH1-4, L1, L_CHG (HAND_EXTENDED).
JLC keeps the 6P USB-C, MT3608, BQ25601 and INA226: ~$21 less setup fee per
order, 87 parts placed. tme.HAND lists the TME parts for them; L1 is the
Ferrocore DJNR6045-100-S (10 uH, Isat 3.1 A, MOQ 5) because TME's
SRN6045-100M is 1000 pcs minimum. lipo keeps its mapping (it wants 4.6 A).

Co-Authored-By: Claude Opus 5.5 <noreply@anthropic.com>
Parts:
- F1, R_SH1: now left out of the parts list
Changed lines of the file:
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@@
 		(body_style 1)
 		(exclude_from_sim no)
-		(in_bom yes)
+		(in_bom no)
 		(on_board yes)
 		(in_pos_files yes)
@@
 		(body_style 1)
 		(exclude_from_sim no)
-		(in_bom yes)
+		(in_bom no)
 		(on_board yes)
 		(in_pos_files yes)
